File: KiCAD/RedPyKeeb.kicad_pcb (KiCad board)
At the start: 2 copper layers, 246 parts, among them K0,0 KEYSW, K0,1 KEYSW, K0,2 KEYSW, K0,3 KEYSW, K0,4 KEYSW, K0,5 KEYSW, K1,0 KEYSW, K1,1 KEYSW, K1,2 KEYSW, K1,3 KEYSW, K1,4 KEYSW, K1,5 KEYSW, K10,0 KEYSW, K10,1 KEYSW, K10,2 KEYSW, K10,3 KEYSW, K10,4 KEYSW, K10,5 KEYSW, K11,0 KEYSW, K11,1 KEYSW, K11,2 KEYSW, K11,3 KEYSW, K11,4 KEYSW, K11,5 KEYSW, K12,0 KEYSW, K12,1 KEYSW, K12,2 KEYSW, K12,3 KEYSW, K12,4 KEYSW, K12,5 KEYSW, K13,1 KEYSW, K13,2 KEYSW, K14,0 KEYSW, K14,1 KEYSW, K14,2 KEYSW, K14,3 KEYSW, K14,4 KEYSW, K14,5 KEYSW, K14,6 KEYSW, K15,0 KEYSW, K15,1 KEYSW, K15,2 KEYSW, K15,3 KEYSW, K15,4 KEYSW, K15,5 KEYSW, K15,6 KEYSW, K16,0 KEYSW, K16,1 KEYSW, K16,2 KEYSW, K16,3 KEYSW, K16,4 KEYSW, K16,5 KEYSW, K16,6 KEYSW, K17,0 KEYSW, K17,1 KEYSW, K17,2 KEYSW, K17,3 KEYSW, K17,4 KEYSW, K17,5 KEYSW, K17,6 KEYSW, K18,0 KEYSW, K18,1 KEYSW, K18,2 KEYSW, K18,3 KEYSW, K18,4 KEYSW, K18,5 KEYSW, K18,6 KEYSW, K19,0 KEYSW, K19,1 KEYSW, K19,2 KEYSW, K19,3 KEYSW, K19,4 KEYSW, K19,5 KEYSW, K19,6 KEYSW, K2,0 KEYSW, K2,1 KEYSW, K2,2 KEYSW, K2,3 KEYSW, K2,4 KEYSW, K2,5 KEYSW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

Commit message: Update KiCAD files
Parts:
- removed D0,10, D0,11, D0,12, D0,13, D0,14, D0,15, D0,16, D0,17, D0,18, D0,19, D0,20, D0,21, D0,22, D0,23, D0,24, D0,25, D0,26, D0,27, D0,28, D0,29, D0,30, D0,31, D0,32, D0,33, D0,34, D0,35, D0,36, D0,37, D0,38, D0,39, D0,40, D0,41, D0,42, D0,43, D0,44, D0,45, D0,46, D0,47, D0,48, D0,49, D0,50, D0,51, D0,52, D0,53, D0,54, D0,55, D0,56, D0,57, D0,58, D0,59, D0,6, D0,60, D0,61, D0,62, D0,63, D0,64, D0,65, D0,66, D0,67, D0,68, D0,69, D0,7, D0,70, D0,71, D0,72, D0,73, D0,74, D0,75, D0,76, D0,77, D0,78, D0,79, D0,8, D0,80, D0,81, D0,82, D0,83, D0,84, D0,85, D0,86, D0,87, D0,88, D0,89, D0,9, D0,90, D0,91, D0,92, D0,93, D0,94, D0,95, D0,96, D0,97, D1,6: D, keyboard_parts:D_SOD123_axial
- removed K12,4, K12,5, K14,2, K14,4, K14,5, K15,2, K15,4, K16,2, K17,2, K18,2, K19,2, K19,5, K4,5, K5,5, K6,5, K7,5: KEYSW, Switch_Keyboard_Kailh:SW_Hotswap_Kailh_1.00u
- added D10,0: D, keyboard_parts:D_SOD123_axial, F.Cu at (298.0, 21.2)
- added D10,1: D, keyboard_parts:D_SOD123_axial, F.Cu at (-21.1, 168.0)
- added D10,2: D, keyboard_parts:D_SOD123_axial, F.Cu at (180.4, 138.5)
- added D10,4: D, keyboard_parts:D_SOD123_axial, F.Cu at (250.4, 67.2)
- added D10,5: D, keyboard_parts:D_SOD123_axial, F.Cu at (250.4, 70.8)
- added D11,0: D, keyboard_parts:D_SOD123_axial, F.Cu at (298.0, 10.4)
- added D11,1: D, keyboard_parts:D_SOD123_axial, F.Cu at (145.3, 168.0)
- added D11,2: D, keyboard_parts:D_SOD123_axial, F.Cu at (180.4, 134.9)
- added D11,3: D, keyboard_parts:D_SOD123_axial, F.Cu at (114.1, 168.0)
- added D11,4: D, keyboard_parts:D_SOD123_axial, F.Cu at (298.0, 14.0)
- added D11,5: D, keyboard_parts:D_SOD123_axial, F.Cu at (145.3, 171.6)
- added D12,0: D, keyboard_parts:D_SOD123_axial, F.Cu at (200.5, 114.7)
- added D12,1: D, keyboard_parts:D_SOD123_axial, F.Cu at (134.9, 168.0)
- added D12,2: D, keyboard_parts:D_SOD123_axial, F.Cu at (200.5, 111.1)
- added D12,3: D, keyboard_parts:D_SOD123_axial, F.Cu at (124.5, 171.6)
- added D13,1: D, keyboard_parts:D_SOD123_axial, F.Cu at (124.5, 168.0)
- added D13,2: D, keyboard_parts:D_SOD123_axial, F.Cu at (114.1, 171.6)
- added D14,0: D, keyboard_parts:D_SOD123_axial, F.Cu at (51.7, 168.0)
- added D14,1: D, keyboard_parts:D_SOD123_axial, F.Cu at (134.9, 171.6)
- added D14,3: D, keyboard_parts:D_SOD123_axial, F.Cu at (298.0, 6.78)
- added D14,66: D, keyboard_parts:D_SOD123_axial, F.Cu at (180.4, 127.7)
- added D15,0: D, keyboard_parts:D_SOD123_axial, F.Cu at (200.5, 107.5)
- added D15,1: D, keyboard_parts:D_SOD123_axial, F.Cu at (190.8, 131.3)
- added D15,3: D, keyboard_parts:D_SOD123_axial, F.Cu at (220.7, 94.6)
- added D15,5: D, keyboard_parts:D_SOD123_axial, F.Cu at (220.7, 91.0)
- added D15,6: D, keyboard_parts:D_SOD123_axial, F.Cu at (220.7, 87.4)
- added D16,0: D, keyboard_parts:D_SOD123_axial, F.Cu at (93.3, 171.6)
- added D16,1: D, keyboard_parts:D_SOD123_axial, F.Cu at (82.9, 168.0)
- added D16,3: D, keyboard_parts:D_SOD123_axial, F.Cu at (82.9, 171.6)
- added D16,4: D, keyboard_parts:D_SOD123_axial, F.Cu at (93.3, 168.0)
- added D16,5: D, keyboard_parts:D_SOD123_axial, F.Cu at (103.7, 168.0)
- added D16,6: D, keyboard_parts:D_SOD123_axial, F.Cu at (103.7, 171.6)
- added D17,0: D, keyboard_parts:D_SOD123_axial, F.Cu at (62.1, 171.6)
- added D17,1: D, keyboard_parts:D_SOD123_axial, F.Cu at (62.1, 168.0)
- added D17,3: D, keyboard_parts:D_SOD123_axial, F.Cu at (72.5, 171.6)
- added D17,4: D, keyboard_parts:D_SOD123_axial, F.Cu at (72.5, 168.0)
- added D17,5: D, keyboard_parts:D_SOD123_axial, F.Cu at (51.7, 171.6)
- added D17,6: D, keyboard_parts:D_SOD123_axial, F.Cu at (41.3, 171.6)
- added D18,0: D, keyboard_parts:D_SOD123_axial, F.Cu at (-10.7, 168.0)
- added D18,1: D, keyboard_parts:D_SOD123_axial, F.Cu at (-21.1, 171.6)
- added D18,3: D, keyboard_parts:D_SOD123_axial, F.Cu at (-0.32, 168.0)
- added D18,4: D, keyboard_parts:D_SOD123_axial, F.Cu at (-0.32, 171.6)
- added D18,5: D, keyboard_parts:D_SOD123_axial, F.Cu at (-10.7, 171.6)
- added D18,6: D, keyboard_parts:D_SOD123_axial, F.Cu at (41.3, 168.0)
- added D19,0: D, keyboard_parts:D_SOD123_axial, F.Cu at (20.5, 168.0)
- added D19,1: D, keyboard_parts:D_SOD123_axial, F.Cu at (30.9, 168.0)
- added D19,3: D, keyboard_parts:D_SOD123_axial, F.Cu at (10.1, 168.0)
- added D19,4: D, keyboard_parts:D_SOD123_axial, F.Cu at (20.5, 171.6)
- added D19,6: D, keyboard_parts:D_SOD123_axial, F.Cu at (10.1, 171.6)
- added D2,2: D, keyboard_parts:D_SOD123_axial, F.Cu at (166.1, 168.0)
- added D2,3: D, keyboard_parts:D_SOD123_axial, F.Cu at (201.2, 132.7)
- added D2,4: D, keyboard_parts:D_SOD123_axial, F.Cu at (295.4, 37.7)
- added D2,5: D, keyboard_parts:D_SOD123_axial, F.Cu at (221.3, 112.6)
- added D20,0: D, keyboard_parts:D_SOD123_axial, F.Cu at (180.4, 131.3)
- added D20,1: D, keyboard_parts:D_SOD123_axial, F.Cu at (30.9, 171.6)
- added D3,2: D, keyboard_parts:D_SOD123_axial, F.Cu at (285.7, 47.1)
- added D3,3: D, keyboard_parts:D_SOD123_axial, F.Cu at (201.2, 125.5)
- added D3,4: D, keyboard_parts:D_SOD123_axial, F.Cu at (221.3, 109.0)
- added D3,5: D, keyboard_parts:D_SOD123_axial, F.Cu at (201.2, 129.1)
- added D4,1: D, keyboard_parts:D_SOD123_axial, F.Cu at (231.1, 101.8)
- added D4,2: D, keyboard_parts:D_SOD123_axial, F.Cu at (221.3, 105.4)
- added D4,3: D, keyboard_parts:D_SOD123_axial, F.Cu at (220.7, 101.8)
- added D4,4: D, keyboard_parts:D_SOD123_axial, F.Cu at (241.5, 87.4)
- added D5,3: D, keyboard_parts:D_SOD123_axial, F.Cu at (180.4, 149.3)
- added D5,4: D, keyboard_parts:D_SOD123_axial, F.Cu at (260.8, 70.8)
- added D6,3: D, keyboard_parts:D_SOD123_axial, F.Cu at (190.8, 134.9)
- added D6,4: D, keyboard_parts:D_SOD123_axial, F.Cu at (180.4, 142.1)
- added D7,3: D, keyboard_parts:D_SOD123_axial, F.Cu at (231.1, 98.2)
- added D7,4: D, keyboard_parts:D_SOD123_axial, F.Cu at (210.9, 114.7)
- added D8,1: D, keyboard_parts:D_SOD123_axial, F.Cu at (295.4, 26.9)
- added D8,2: D, keyboard_parts:D_SOD123_axial, F.Cu at (155.7, 168.0)
- added D8,3: D, keyboard_parts:D_SOD123_axial, F.Cu at (275.3, 47.1)
- added D8,4: D, keyboard_parts:D_SOD123_axial, F.Cu at (231.1, 91.0)
- added D8,5: D, keyboard_parts:D_SOD123_axial, F.Cu at (231.1, 87.4)
- added D9,1: D, keyboard_parts:D_SOD123_axial, F.Cu at (210.9, 107.5)
- added D9,2: D, keyboard_parts:D_SOD123_axial, F.Cu at (210.9, 111.1)
- added D9,3: D, keyboard_parts:D_SOD123_axial, F.Cu at (200.5, 121.9)
- added D9,4: D, keyboard_parts:D_SOD123_axial, F.Cu at (221.3, 116.2)
- added D9,5: D, keyboard_parts:D_SOD123_axial, F.Cu at (190.8, 127.7)
- added J0: Conn_01x04, Connector_JST:JST_EH_S4B-EH_1x04_P2.50mm_Horizontal, F.Cu at (1.29, 214.1)
- added J1: Conn_01x04, Connector_JST:JST_EH_S4B-EH_1x04_P2.50mm_Horizontal, F.Cu at (1.29, 203.7)
- added K20,0: KEYSW, Switch_Keyboard_Kailh:SW_Hotswap_Kailh_1.00u, F.Cu at (147.9, -5.09)
- added K20,1: KEYSW, Switch_Keyboard_Kailh:SW_Hotswap_Kailh_1.00u, F.Cu at (33.6, 75.5)
- added LD0,0: APA102-2020, CrumpPrints:APA102_hand_solder, F.Cu at (413.6, 19.0)
- added LD0,1: APA102-2020, CrumpPrints:APA102_hand_solder, F.Cu at (358.2, 3.83)
- added LD0,2: APA102-2020, CrumpPrints:APA102_hand_solder, F.Cu at (395.1, 34.2)
- added LD0,3: APA102-2020, CrumpPrints:APA102_hand_solder, F.Cu at (315.2, -3.77)
- added LD0,4: APA102-2020, CrumpPrints:APA102_hand_solder, F.Cu at (321.3, -11.4)
- added LD0,5: APA102-2020, CrumpPrints:APA102_hand_solder, F.Cu at (401.3, 34.2)
- added LD1,0: APA102-2020, CrumpPrints:APA102_hand_solder, F.Cu at (327.5, -3.77)
- added LD1,1: APA102-2020, CrumpPrints:APA102_hand_solder, F.Cu at (315.2, 3.83)
- added LD1,2: APA102-2020, CrumpPrints:APA102_hand_solder, F.Cu at (321.3, -3.77)
- added LD1,3: APA102-2020, CrumpPrints:APA102_hand_solder, F.Cu at (315.2, 11.4)
- added LD1,4: APA102-2020, CrumpPrints:APA102_hand_solder, F.Cu at (321.3, 3.83)
- added LD1,5: APA102-2020, CrumpPrints:APA102_hand_solder, F.Cu at (327.5, -11.4)
- added LD10,0: APA102-2020, CrumpPrints:APA102_hand_solder, F.Cu at (389.0, -11.4)
- added LD10,1: APA102-2020, CrumpPrints:APA102_hand_solder, F.Cu at (376.7, -3.77)
- added LD10,2: APA102-2020, CrumpPrints:APA102_hand_solder, F.Cu at (382.8, -11.4)
- added LD10,3: APA102-2020, CrumpPrints:APA102_hand_solder, F.Cu at (395.1, 3.83)
- added LD10,4: APA102-2020, CrumpPrints:APA102_hand_solder, F.Cu at (352.1, 26.6)
- added LD10,5: APA102-2020, CrumpPrints:APA102_hand_solder, F.Cu at (358.2, 19.0)
- added LD11,0: APA102-2020, CrumpPrints:APA102_hand_solder, F.Cu at (376.7, 3.83)
- added LD11,1: APA102-2020, CrumpPrints:APA102_hand_solder, F.Cu at (382.8, -3.77)
- added LD11,2: APA102-2020, CrumpPrints:APA102_hand_solder, F.Cu at (358.2, 26.6)
- added LD11,3: APA102-2020, CrumpPrints:APA102_hand_solder, F.Cu at (364.4, 19.0)
- added LD11,4: APA102-2020, CrumpPrints:APA102_hand_solder, F.Cu at (345.9, 34.2)
- added LD11,5: APA102-2020, CrumpPrints:APA102_hand_solder, F.Cu at (370.5, 11.4)
- added LD12,0: APA102-2020, CrumpPrints:APA102_hand_solder, F.Cu at (352.1, 34.2)
- added LD12,1: APA102-2020, CrumpPrints:APA102_hand_solder, F.Cu at (389.0, -3.77)
- added LD12,2: APA102-2020, CrumpPrints:APA102_hand_solder, F.Cu at (364.4, 26.6)
- added LD12,3: APA102-2020, CrumpPrints:APA102_hand_solder, F.Cu at (395.1, -11.4)
- added LD13,0: APA102-2020, CrumpPrints:APA102_hand_solder, F.Cu at (370.5, 3.83)
- added LD13,1: APA102-2020, CrumpPrints:APA102_hand_solder, F.Cu at (370.5, 19.0)
- added LD13,2: APA102-2020, CrumpPrints:APA102_hand_solder, F.Cu at (376.7, 11.4)
- added LD14,0: APA102-2020, CrumpPrints:APA102_hand_solder, F.Cu at (389.0, 3.83)
- added LD14,1: APA102-2020, CrumpPrints:APA102_hand_solder, F.Cu at (395.1, -3.77)
- added LD14,3: APA102-2020, CrumpPrints:APA102_hand_solder, F.Cu at (382.8, 3.83)
- added LD14,6: APA102-2020, CrumpPrints:APA102_hand_solder, F.Cu at (358.2, 34.2)
- added LD15,0: APA102-2020, CrumpPrints:APA102_hand_solder, F.Cu at (401.3, -3.77)
- added LD15,1: APA102-2020, CrumpPrints:APA102_hand_solder, F.Cu at (382.8, 11.4)
- added LD15,3: APA102-2020, CrumpPrints:APA102_hand_solder, F.Cu at (370.5, 26.6)
- added LD15,5: APA102-2020, CrumpPrints:APA102_hand_solder, F.Cu at (376.7, 19.0)
- added LD15,6: APA102-2020, CrumpPrints:APA102_hand_solder, F.Cu at (364.4, 34.2)
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Connections:
- net I2C_SCL1 renamed Net-(U0-Pad20)
- net I2C_SDA1 renamed Net-(U0-Pad19)
- net KEY_COL10 renamed Net-(U0-Pad16)
- net KEY_COL11 renamed Net-(U0-Pad17)
- net KEY_COL12 renamed Net-(U0-Pad22)
- net KEY_COL13 renamed Net-(U0-Pad21)
- net KEY_COL7 renamed Net-(U0-Pad12)
- net KEY_COL8 renamed Net-(U0-Pad14)
- net KEY_COL9 renamed Net-(U0-Pad15)
- D0,2 pad 1: Net-(D0,10-Pad1) -> Net-(D0,2-Pad1)
- D0,3 pad 1: Net-(D0,17-Pad1) -> Net-(D0,3-Pad1)
- D0,4 pad 1: Net-(D0,11-Pad1) -> Net-(D0,4-Pad1)
- D0,5 pad 1: Net-(D0,11-Pad1) -> Net-(D0,5-Pad1)
- D1,1 pad 1: Net-(D0,10-Pad1) -> Net-(D0,1-Pad1)
- D1,2 pad 1: Net-(D0,17-Pad1) -> Net-(D0,2-Pad1)
- D1,3 pad 1: Net-(D0,1-Pad1) -> Net-(D0,3-Pad1)
- D1,4 pad 1: Net-(D0,0-Pad1) -> Net-(D0,4-Pad1)
- D1,5 pad 1: Net-(D0,10-Pad1) -> Net-(D0,5-Pad1)
- D10,3 pad 1: Net-(D0,1-Pad1) -> Net-(D0,3-Pad1)
- D2,1 pad 1: Net-(D0,0-Pad1) -> Net-(D0,1-Pad1)
- D3,1 pad 1: Net-(D0,0-Pad1) -> Net-(D0,1-Pad1)
- D5,1 pad 1: Net-(D5,1-Pad1) -> Net-(D0,1-Pad1)
- D5,2 pad 1: Net-(D5,1-Pad1) -> Net-(D0,2-Pad1)
- D6,1 pad 1: Net-(D5,1-Pad1) -> Net-(D0,1-Pad1)
- D6,2 pad 1: Net-(D5,1-Pad1) -> Net-(D0,2-Pad1)
- D7,1 pad 1: Net-(D5,1-Pad1) -> Net-(D0,1-Pad1)
- D7,2 pad 1: Net-(D5,1-Pad1) -> Net-(D0,2-Pad1)
- K0,1 pad 2: Net-(D0,2-Pad2) -> Net-(D0,1-Pad2)
- K0,2 pad 2: Net-(D0,3-Pad2) -> Net-(D0,2-Pad2)
- K0,3 pad 2: Net-(D0,1-Pad2) -> Net-(D0,3-Pad2)
- K0,5 pad 2: Net-(D0,7-Pad2) -> Net-(D0,5-Pad2)
- K1,4 pad 2: Net-(D0,11-Pad2) -> Net-(D1,4-Pad2)
- K1,5 pad 2: Net-(D0,12-Pad2) -> Net-(D1,5-Pad2)
- K10,0 pad 2: Net-(D1,4-Pad2) -> Net-(D10,0-Pad2)
- K10,1 pad 2: Net-(D1,5-Pad2) -> Net-(D10,1-Pad2)
- K10,4 pad 2: Net-(D0,5-Pad2) -> Net-(D10,4-Pad2)
- K11,0 pad 2: Net-(D2,1-Pad2) -> Net-(D11,0-Pad2)
- K12,0 pad 2: Net-(D3,1-Pad2) -> Net-(D12,0-Pad2)
- K14,0 pad 2: Net-(D5,1-Pad2) -> Net-(D14,0-Pad2)
- K15,0 pad 2: Net-(D6,1-Pad2) -> Net-(D15,0-Pad2)
- K16,0 pad 2: Net-(D7,1-Pad2) -> Net-(D16,0-Pad2)
- K17,0 pad 2: Net-(D5,2-Pad2) -> Net-(D17,0-Pad2)
- K18,0 pad 2: Net-(D6,2-Pad2) -> Net-(D18,0-Pad2)
- K19,0 pad 2: Net-(D7,2-Pad2) -> Net-(D19,0-Pad2)
- K2,1 pad 2: Net-(D0,8-Pad2) -> Net-(D2,1-Pad2)
- K3,1 pad 2: Net-(D0,16-Pad2) -> Net-(D3,1-Pad2)
- K5,1 pad 2: Net-(D0,26-Pad2) -> Net-(D5,1-Pad2)
- K5,2 pad 2: Net-(D0,27-Pad2) -> Net-(D5,2-Pad2)
- K6,1 pad 2: Net-(D0,31-Pad2) -> Net-(D6,1-Pad2)
- K6,2 pad 2: Net-(D0,32-Pad2) -> Net-(D6,2-Pad2)
- K7,1 pad 2: Net-(D0,36-Pad2) -> Net-(D7,1-Pad2)
- K7,2 pad 2: Net-(D0,37-Pad2) -> Net-(D7,2-Pad2)
- U0 pad 10: KEY_COL5 -> IO_INT3
- U0 pad 11: KEY_COL6 -> Net-(U0-Pad11)
- U0 pad 25: KEY_ROW0 -> Net-(U0-Pad25)
- U0 pad 26: KEY_ROW1 -> Net-(U0-Pad26)
- U0 pad 27: KEY_ROW2 -> Net-(U0-Pad27)
- U0 pad 29: KEY_ROW3 -> Net-(U0-Pad29)
- U0 pad 31: KEY_ROW4 -> Net-(U0-Pad31)
- U0 pad 32: KEY_ROW5 -> Net-(U0-Pad32)
- U0 pad 39: Net-(U0-Pad39) -> MAIN_VBUS
- U0 pad 4: KEY_COL0 -> Net-(U0-Pad4)
- U0 pad 40: Net-(U0-Pad39) -> Net-(U0-Pad40)
- U0 pad 5: KEY_COL1 -> Net-(U0-Pad5)
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Routing:
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
Commit message: Update KiCAD files
Parts:
- added C1: 0805B104K100CT, Capacitors_SMD:C_0805_HandSoldering, F.Cu at (400.9, 41.8)
- added C2: 0805B104K100CT, Capacitors_SMD:C_0805_HandSoldering, F.Cu at (400.9, 39.0)
- added C3: 0805B104K100CT, Capacitors_SMD:C_0805_HandSoldering, F.Cu at (406.5, 39.0)
- added C6: EEE-FK1A102AL, Capacitor_SMD:CP_Elec_10x10, F.Cu at (28.4, 228.1)
- added U999: TL750M05CKTTR, Package_TO_SOT_SMD:TO-263-3_TabPin2, F.Cu at (29.9, 216.0)
- U0: footprint MCU_RaspberryPi_and_Boards:RPi_Pico_SMD_TH -> Custom_pico:RPi_Pico_SMD_TH
- moved LD18,0 454.2 mm to (48.8, 266.8)
- moved U3 441.1 mm to (415.9, 27.9)
- moved LD16,1 439.5 mm to (73.4, 266.8)
- moved LD15,0 434.7 mm to (61.1, 266.8)
- moved LD0,0 428.6 mm to (38.2, 226.0)
- moved LD16,3 425.2 mm to (79.5, 266.8)
- moved LD7,2 421.7 mm to (24.2, 237.8)
- moved LD5,5 421.2 mm to (30.3, 260.6)
- moved LD10,1 420.4 mm to (54.9, 266.8)
- moved LD8,4 420.4 mm to (54.9, 259.2)
- moved LD5,0 418.6 mm to (36.5, 256.4)
- moved J0 417.1 mm to (387.1, 55.7)
- moved J1 417.1 mm to (387.1, 45.3)
- moved U0 416.7 mm to (361.1, 70.2)
- moved LD18,4 415.6 mm to (85.7, 266.8)
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Connections:
- LD0,0 pad 6: Net-(LD0,0-Pad6) -> GNDPWR
- LD0,1 pad 1: Net-(LD0,1-Pad1) -> Net-(LD0,0-Pad1)
- LD0,1 pad 6: Net-(LD0,1-Pad6) -> GNDPWR
- LD0,2 pad 1: Net-(LD0,2-Pad1) -> Net-(LD0,0-Pad1)
- LD0,2 pad 6: Net-(LD0,2-Pad6) -> GNDPWR
- LD0,3 pad 1: Net-(LD0,3-Pad1) -> Net-(LD0,0-Pad1)
- LD0,3 pad 6: Net-(LD0,3-Pad6) -> GNDPWR
- LD0,4 pad 1: Net-(LD0,4-Pad1) -> Net-(LD0,0-Pad1)
- LD0,4 pad 6: Net-(LD0,4-Pad6) -> GNDPWR
- LD0,5 pad 1: Net-(LD0,5-Pad1) -> Net-(LD0,0-Pad1)
- LD0,5 pad 6: Net-(LD0,5-Pad6) -> GNDPWR
- LD1,0 pad 6: Net-(LD0,0-Pad6) -> GNDPWR
- LD1,1 pad 1: Net-(LD0,1-Pad1) -> Net-(LD0,0-Pad1)
- LD1,1 pad 6: Net-(LD0,1-Pad6) -> GNDPWR
- LD1,2 pad 1: Net-(LD0,2-Pad1) -> Net-(LD0,0-Pad1)
- LD1,2 pad 6: Net-(LD0,2-Pad6) -> GNDPWR
- LD1,3 pad 1: Net-(LD0,3-Pad1) -> Net-(LD0,0-Pad1)
- LD1,3 pad 6: Net-(LD0,3-Pad6) -> GNDPWR
- LD1,4 pad 1: Net-(LD0,4-Pad1) -> Net-(LD0,0-Pad1)
- LD1,4 pad 6: Net-(LD0,4-Pad6) -> GNDPWR
- LD1,5 pad 1: Net-(LD0,5-Pad1) -> Net-(LD0,0-Pad1)
- LD1,5 pad 6: Net-(LD0,5-Pad6) -> GNDPWR
- LD10,0 pad 6: Net-(LD0,0-Pad6) -> GNDPWR
- LD10,1 pad 1: Net-(LD0,1-Pad1) -> Net-(LD0,0-Pad1)
- LD10,1 pad 6: Net-(LD0,1-Pad6) -> GNDPWR
- LD10,2 pad 1: Net-(LD0,2-Pad1) -> Net-(LD0,0-Pad1)
- LD10,2 pad 6: Net-(LD0,2-Pad6) -> GNDPWR
- LD10,3 pad 1: Net-(LD0,3-Pad1) -> Net-(LD0,0-Pad1)
- LD10,3 pad 6: Net-(LD0,3-Pad6) -> GNDPWR
- LD10,4 pad 1: Net-(LD0,4-Pad1) -> Net-(LD0,0-Pad1)
- LD10,4 pad 6: Net-(LD0,4-Pad6) -> GNDPWR
- LD10,5 pad 1: Net-(LD0,5-Pad1) -> Net-(LD0,0-Pad1)
- LD10,5 pad 6: Net-(LD0,5-Pad6) -> GNDPWR
- LD11,0 pad 6: Net-(LD0,0-Pad6) -> GNDPWR
- LD11,1 pad 1: Net-(LD0,1-Pad1) -> Net-(LD0,0-Pad1)
- LD11,1 pad 6: Net-(LD0,1-Pad6) -> GNDPWR
- LD11,2 pad 1: Net-(LD0,2-Pad1) -> Net-(LD0,0-Pad1)
- LD11,2 pad 6: Net-(LD0,2-Pad6) -> GNDPWR
- LD11,3 pad 1: Net-(LD0,3-Pad1) -> Net-(LD0,0-Pad1)
- LD11,3 pad 6: Net-(LD0,3-Pad6) -> GNDPWR
- LD11,4 pad 1: Net-(LD0,4-Pad1) -> Net-(LD0,0-Pad1)
- LD11,4 pad 6: Net-(LD0,4-Pad6) -> GNDPWR
- LD11,5 pad 1: Net-(LD0,5-Pad1) -> Net-(LD0,0-Pad1)
- LD11,5 pad 6: Net-(LD0,5-Pad6) -> GNDPWR
- LD12,0 pad 6: Net-(LD0,0-Pad6) -> GNDPWR
- LD12,1 pad 1: Net-(LD0,1-Pad1) -> Net-(LD0,0-Pad1)
- LD12,1 pad 6: Net-(LD0,1-Pad6) -> GNDPWR
- LD12,2 pad 1: Net-(LD0,2-Pad1) -> Net-(LD0,0-Pad1)
- LD12,2 pad 6: Net-(LD0,2-Pad6) -> GNDPWR
- LD12,3 pad 1: Net-(LD0,3-Pad1) -> Net-(LD0,0-Pad1)
- LD12,3 pad 6: Net-(LD0,3-Pad6) -> GNDPWR
- LD13,0 pad 6: Net-(LD0,0-Pad6) -> GNDPWR
- LD13,1 pad 1: Net-(LD0,1-Pad1) -> Net-(LD0,0-Pad1)
- LD13,1 pad 6: Net-(LD0,1-Pad6) -> GNDPWR
- LD13,2 pad 1: Net-(LD0,2-Pad1) -> Net-(LD0,0-Pad1)
- LD13,2 pad 6: Net-(LD0,2-Pad6) -> GNDPWR
- LD14,0 pad 6: Net-(LD0,0-Pad6) -> GNDPWR
- LD14,1 pad 1: Net-(LD0,1-Pad1) -> Net-(LD0,0-Pad1)
- LD14,1 pad 6: Net-(LD0,1-Pad6) -> GNDPWR
- LD14,3 pad 1: Net-(LD0,3-Pad1) -> Net-(LD0,0-Pad1)
- LD14,3 pad 6: Net-(LD0,3-Pad6) -> GNDPWR
- LD14,6 pad 1: Net-(LD14,6-Pad1) -> Net-(LD0,0-Pad1)
- LD14,6 pad 6: Net-(LD14,6-Pad6) -> GNDPWR
- LD15,0 pad 6: Net-(LD0,0-Pad6) -> GNDPWR
- LD15,1 pad 1: Net-(LD0,1-Pad1) -> Net-(LD0,0-Pad1)
- LD15,1 pad 6: Net-(LD0,1-Pad6) -> GNDPWR
- LD15,3 pad 1: Net-(LD0,3-Pad1) -> Net-(LD0,0-Pad1)
- LD15,3 pad 6: Net-(LD0,3-Pad6) -> GNDPWR
- LD15,5 pad 1: Net-(LD0,5-Pad1) -> Net-(LD0,0-Pad1)
- LD15,5 pad 6: Net-(LD0,5-Pad6) -> GNDPWR
- LD15,6 pad 1: Net-(LD14,6-Pad1) -> Net-(LD0,0-Pad1)
- LD15,6 pad 6: Net-(LD14,6-Pad6) -> GNDPWR
- LD16,0 pad 6: Net-(LD0,0-Pad6) -> GNDPWR
- LD16,1 pad 1: Net-(LD0,1-Pad1) -> Net-(LD0,0-Pad1)
- LD16,1 pad 6: Net-(LD0,1-Pad6) -> GNDPWR
- LD16,3 pad 1: Net-(LD0,3-Pad1) -> Net-(LD0,0-Pad1)
- LD16,3 pad 6: Net-(LD0,3-Pad6) -> GNDPWR
- LD16,4 pad 1: Net-(LD0,4-Pad1) -> Net-(LD0,0-Pad1)
- LD16,4 pad 6: Net-(LD0,4-Pad6) -> GNDPWR
- LD16,5 pad 1: Net-(LD0,5-Pad1) -> Net-(LD0,0-Pad1)
- LD16,5 pad 6: Net-(LD0,5-Pad6) -> GNDPWR
- LD16,6 pad 1: Net-(LD14,6-Pad1) -> Net-(LD0,0-Pad1)
- LD16,6 pad 6: Net-(LD14,6-Pad6) -> GNDPWR
- LD17,0 pad 6: Net-(LD0,0-Pad6) -> GNDPWR
- LD17,1 pad 1: Net-(LD0,1-Pad1) -> Net-(LD0,0-Pad1)
- LD17,1 pad 6: Net-(LD0,1-Pad6) -> GNDPWR
- LD17,3 pad 1: Net-(LD0,3-Pad1) -> Net-(LD0,0-Pad1)
- LD17,3 pad 6: Net-(LD0,3-Pad6) -> GNDPWR
- LD17,4 pad 1: Net-(LD0,4-Pad1) -> Net-(LD0,0-Pad1)
- LD17,4 pad 6: Net-(LD0,4-Pad6) -> GNDPWR
- LD17,5 pad 1: Net-(LD0,5-Pad1) -> Net-(LD0,0-Pad1)
- LD17,5 pad 6: Net-(LD0,5-Pad6) -> GNDPWR
- LD17,6 pad 1: Net-(LD14,6-Pad1) -> Net-(LD0,0-Pad1)
- LD17,6 pad 6: Net-(LD14,6-Pad6) -> GNDPWR
- LD18,0 pad 6: Net-(LD0,0-Pad6) -> GNDPWR
- LD18,1 pad 1: Net-(LD0,1-Pad1) -> Net-(LD0,0-Pad1)
- LD18,1 pad 6: Net-(LD0,1-Pad6) -> GNDPWR
- LD18,3 pad 1: Net-(LD0,3-Pad1) -> Net-(LD0,0-Pad1)
- LD18,3 pad 6: Net-(LD0,3-Pad6) -> GNDPWR
- LD18,4 pad 1: Net-(LD0,4-Pad1) -> Net-(LD0,0-Pad1)
- LD18,4 pad 6: Net-(LD0,4-Pad6) -> GNDPWR
- LD18,5 pad 1: Net-(LD0,5-Pad1) -> Net-(LD0,0-Pad1)
- LD18,5 pad 6: Net-(LD0,5-Pad6) -> GNDPWR
- LD18,6 pad 1: Net-(LD14,6-Pad1) -> Net-(LD0,0-Pad1)
- LD18,6 pad 6: Net-(LD14,6-Pad6) -> GNDPWR
- LD19,0 pad 6: Net-(LD0,0-Pad6) -> GNDPWR
- LD19,1 pad 1: Net-(LD0,1-Pad1) -> Net-(LD0,0-Pad1)
- LD19,1 pad 6: Net-(LD0,1-Pad6) -> GNDPWR
- LD19,3 pad 1: Net-(LD0,3-Pad1) -> Net-(LD0,0-Pad1)
- LD19,3 pad 6: Net-(LD0,3-Pad6) -> GNDPWR
- LD19,4 pad 1: Net-(LD0,4-Pad1) -> Net-(LD0,0-Pad1)
- LD19,4 pad 6: Net-(LD0,4-Pad6) -> GNDPWR
- LD19,6 pad 1: Net-(LD14,6-Pad1) -> Net-(LD0,0-Pad1)
- LD19,6 pad 6: Net-(LD14,6-Pad6) -> GNDPWR
- LD2,0 pad 6: Net-(LD0,0-Pad6) -> GNDPWR
- LD2,1 pad 1: Net-(LD0,1-Pad1) -> Net-(LD0,0-Pad1)
- LD2,1 pad 6: Net-(LD0,1-Pad6) -> GNDPWR
- LD2,2 pad 1: Net-(LD0,2-Pad1) -> Net-(LD0,0-Pad1)
- LD2,2 pad 6: Net-(LD0,2-Pad6) -> GNDPWR
- LD2,3 pad 1: Net-(LD0,3-Pad1) -> Net-(LD0,0-Pad1)
- LD2,3 pad 6: Net-(LD0,3-Pad6) -> GNDPWR
- LD2,4 pad 1: Net-(LD0,4-Pad1) -> Net-(LD0,0-Pad1)
- LD2,4 pad 6: Net-(LD0,4-Pad6) -> GNDPWR
- LD2,5 pad 1: Net-(LD0,5-Pad1) -> Net-(LD0,0-Pad1)
- LD2,5 pad 6: Net-(LD0,5-Pad6) -> GNDPWR
- LD20,0 pad 6: Net-(LD0,0-Pad6) -> GNDPWR
- LD20,1 pad 1: Net-(LD0,1-Pad1) -> Net-(LD0,0-Pad1)
- LD20,1 pad 6: Net-(LD0,1-Pad6) -> GNDPWR
- LD20,4 pad 1: Net-(LD0,4-Pad1) -> Net-(LD0,0-Pad1)
- LD20,4 pad 6: Net-(LD0,4-Pad6) -> GNDPWR
- LD20,6 pad 1: Net-(LD14,6-Pad1) -> Net-(LD0,0-Pad1)
- LD20,6 pad 6: Net-(LD14,6-Pad6) -> GNDPWR
- LD3,0 pad 6: Net-(LD0,0-Pad6) -> GNDPWR
- LD3,1 pad 1: Net-(LD0,1-Pad1) -> Net-(LD0,0-Pad1)
- LD3,1 pad 6: Net-(LD0,1-Pad6) -> GNDPWR
- LD3,2 pad 1: Net-(LD0,2-Pad1) -> Net-(LD0,0-Pad1)
- LD3,2 pad 6: Net-(LD0,2-Pad6) -> GNDPWR
- LD3,3 pad 1: Net-(LD0,3-Pad1) -> Net-(LD0,0-Pad1)
- LD3,3 pad 6: Net-(LD0,3-Pad6) -> GNDPWR
- LD3,4 pad 1: Net-(LD0,4-Pad1) -> Net-(LD0,0-Pad1)
- LD3,4 pad 6: Net-(LD0,4-Pad6) -> GNDPWR
- LD3,5 pad 1: Net-(LD0,5-Pad1) -> Net-(LD0,0-Pad1)
- LD3,5 pad 6: Net-(LD0,5-Pad6) -> GNDPWR
- LD4,0 pad 6: Net-(LD0,0-Pad6) -> GNDPWR
- LD4,1 pad 1: Net-(LD0,1-Pad1) -> Net-(LD0,0-Pad1)
- LD4,1 pad 6: Net-(LD0,1-Pad6) -> GNDPWR
- LD4,2 pad 1: Net-(LD0,2-Pad1) -> Net-(LD0,0-Pad1)
- LD4,2 pad 6: Net-(LD0,2-Pad6) -> GNDPWR
- LD4,3 pad 1: Net-(LD0,3-Pad1) -> Net-(LD0,0-Pad1)
- LD4,3 pad 6: Net-(LD0,3-Pad6) -> GNDPWR
- LD4,4 pad 1: Net-(LD0,4-Pad1) -> Net-(LD0,0-Pad1)
- LD4,4 pad 6: Net-(LD0,4-Pad6) -> GNDPWR
- LD4,5 pad 1: Net-(LD0,5-Pad1) -> Net-(LD0,0-Pad1)
- LD4,5 pad 6: Net-(LD0,5-Pad6) -> GNDPWR
- LD5,0 pad 6: Net-(LD0,0-Pad6) -> GNDPWR
- LD5,1 pad 1: Net-(LD0,1-Pad1) -> Net-(LD0,0-Pad1)
- LD5,1 pad 6: Net-(LD0,1-Pad6) -> GNDPWR
- LD5,2 pad 1: Net-(LD0,2-Pad1) -> Net-(LD0,0-Pad1)
- LD5,2 pad 6: Net-(LD0,2-Pad6) -> GNDPWR
- LD5,3 pad 1: Net-(LD0,3-Pad1) -> Net-(LD0,0-Pad1)
- LD5,3 pad 6: Net-(LD0,3-Pad6) -> GNDPWR
- LD5,4 pad 1: Net-(LD0,4-Pad1) -> Net-(LD0,0-Pad1)
- LD5,4 pad 6: Net-(LD0,4-Pad6) -> GNDPWR
- LD5,5 pad 1: Net-(LD0,5-Pad1) -> Net-(LD0,0-Pad1)
- LD5,5 pad 6: Net-(LD0,5-Pad6) -> GNDPWR
- LD6,0 pad 6: Net-(LD0,0-Pad6) -> GNDPWR
- LD6,1 pad 1: Net-(LD0,1-Pad1) -> Net-(LD0,0-Pad1)
- LD6,1 pad 6: Net-(LD0,1-Pad6) -> GNDPWR
- LD6,2 pad 1: Net-(LD0,2-Pad1) -> Net-(LD0,0-Pad1)
- LD6,2 pad 6: Net-(LD0,2-Pad6) -> GNDPWR
- LD6,3 pad 1: Net-(LD0,3-Pad1) -> Net-(LD0,0-Pad1)
- LD6,3 pad 6: Net-(LD0,3-Pad6) -> GNDPWR
- LD6,4 pad 1: Net-(LD0,4-Pad1) -> Net-(LD0,0-Pad1)
- LD6,4 pad 6: Net-(LD0,4-Pad6) -> GNDPWR
- LD6,5 pad 1: Net-(LD0,5-Pad1) -> Net-(LD0,0-Pad1)
- LD6,5 pad 6: Net-(LD0,5-Pad6) -> GNDPWR
- LD7,0 pad 6: Net-(LD0,0-Pad6) -> GNDPWR
- LD7,1 pad 1: Net-(LD0,1-Pad1) -> Net-(LD0,0-Pad1)
- LD7,1 pad 6: Net-(LD0,1-Pad6) -> GNDPWR
- LD7,2 pad 1: Net-(LD0,2-Pad1) -> Net-(LD0,0-Pad1)
- LD7,2 pad 6: Net-(LD0,2-Pad6) -> GNDPWR
- LD7,3 pad 1: Net-(LD0,3-Pad1) -> Net-(LD0,0-Pad1)
- LD7,3 pad 6: Net-(LD0,3-Pad6) -> GNDPWR
- LD7,4 pad 1: Net-(LD0,4-Pad1) -> Net-(LD0,0-Pad1)
- LD7,4 pad 6: Net-(LD0,4-Pad6) -> GNDPWR
- LD7,5 pad 1: Net-(LD0,5-Pad1) -> Net-(LD0,0-Pad1)
- LD7,5 pad 6: Net-(LD0,5-Pad6) -> GNDPWR
- LD8,0 pad 6: Net-(LD0,0-Pad6) -> GNDPWR
- LD8,1 pad 1: Net-(LD0,1-Pad1) -> Net-(LD0,0-Pad1)
- LD8,1 pad 6: Net-(LD0,1-Pad6) -> GNDPWR
- LD8,2 pad 1: Net-(LD0,2-Pad1) -> Net-(LD0,0-Pad1)
- LD8,2 pad 6: Net-(LD0,2-Pad6) -> GNDPWR
- LD8,3 pad 1: Net-(LD0,3-Pad1) -> Net-(LD0,0-Pad1)
- LD8,3 pad 6: Net-(LD0,3-Pad6) -> GNDPWR
- LD8,4 pad 1: Net-(LD0,4-Pad1) -> Net-(LD0,0-Pad1)
- LD8,4 pad 6: Net-(LD0,4-Pad6) -> GNDPWR
- LD8,5 pad 1: Net-(LD0,5-Pad1) -> Net-(LD0,0-Pad1)
- LD8,5 pad 6: Net-(LD0,5-Pad6) -> GNDPWR
- LD9,0 pad 6: Net-(LD0,0-Pad6) -> GNDPWR
- LD9,1 pad 1: Net-(LD0,1-Pad1) -> Net-(LD0,0-Pad1)
- LD9,1 pad 6: Net-(LD0,1-Pad6) -> GNDPWR
- LD9,2 pad 1: Net-(LD0,2-Pad1) -> Net-(LD0,0-Pad1)
- LD9,2 pad 6: Net-(LD0,2-Pad6) -> GNDPWR
- LD9,3 pad 1: Net-(LD0,3-Pad1) -> Net-(LD0,0-Pad1)
- LD9,3 pad 6: Net-(LD0,3-Pad6) -> GNDPWR
- LD9,4 pad 1: Net-(LD0,4-Pad1) -> Net-(LD0,0-Pad1)
- LD9,4 pad 6: Net-(LD0,4-Pad6) -> GNDPWR
- LD9,5 pad 1: Net-(LD0,5-Pad1) -> Net-(LD0,0-Pad1)
- LD9,5 pad 6: Net-(LD0,5-Pad6) -> GNDPWR
- U0 pad 38: GNDPWR -> Net-(U0-Pad38)

Commit message: Update KiCAD files and README
Parts:
- added LD17,7: APA102-2020, CrumpPrints:APA102_hand_solder, F.Cu at (96.3, 256.0)
- added LD18,7: APA102-2020, CrumpPrints:APA102_hand_solder, F.Cu at (122.7, 233.2)
- added LD19,7: APA102-2020, CrumpPrints:APA102_hand_solder, F.Cu at (127.1, 240.8)
- added LD20,7: APA102-2020, CrumpPrints:APA102_hand_solder, F.Cu at (120.9, 248.4)
- moved K16,4 296.5 mm to (294.3, 52.7)
- moved K16,5 270.9 mm to (76.0, 153.5)
- moved D9,0 244.8 mm to (272.6, 135.8)
- moved K17,4 233.1 mm to (219.9, 32.6)
- moved D14,66 231.9 mm to (186.8, 209.2)
- moved K7,3 217.1 mm to (280.4, 32.6)
- moved K17,5 215.9 mm to (55.8, 173.6)
- moved K3,2 201.8 mm to (340.8, 32.6)
- moved K0,2 199.9 mm to (334.6, 52.7)
- moved D12,1 199.1 mm to (272.6, 128.6)
- moved D8,4 196.3 mm to (347.3, 68.2)
- moved D12,3 192.9 mm to (93.2, 209.2)
- moved D9,2 191.1 mm to (41.2, 205.6)
- moved D2,3 183.7 mm to (347.3, 75.4)
- moved K15,6 175.3 mm to (35.7, 133.3)
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Connections:
- U3 pad 28: Net-(U3-Pad28) -> LED_SDA_ROW7
- U3 pad 8: Net-(U3-Pad8) -> LED_SCL_ROW7

Commit message: Update KiCAD files
Parts:
- K0,2: footprint Switch_Keyboard_Kailh:SW_Hotswap_Kailh_1.00u -> Switch_Keyboard_Kailh:SW_Hotswap_Kailh_1.50u
- K0,3: footprint Switch_Keyboard_Kailh:SW_Hotswap_Kailh_1.00u -> Switch_Keyboard_Kailh:SW_Hotswap_Kailh_1.75u
- K0,4: footprint Switch_Keyboard_Kailh:SW_Hotswap_Kailh_1.00u -> Switch_Keyboard_Kailh:SW_Hotswap_Kailh_2.25u
- K17,6: footprint Switch_Keyboard_Kailh:SW_Hotswap_Kailh_1.00u -> Switch_Keyboard_Kailh:SW_Hotswap_Kailh_2.00u
- K19,4, K19,6: footprint Switch_Keyboard_Kailh:SW_Hotswap_Kailh_1.00u -> Switch_Keyboard_Kailh:SW_Hotswap_Kailh_2.00u_Rotated
- moved D9,2 358.4 mm to (353.8, 30.4)
- moved K0,2 286.6 mm to (53.5, 108.4)
- moved D14,0 280.3 mm to (117.3, 200.9)
- moved D10,0 246.9 mm to (158.9, 204.5)
- moved K10,4 246.2 mm to (257.9, 27.8)
- moved D10,1 242.4 mm to (158.9, 200.9)
- moved D12,1 241.5 mm to (44.5, 208.1)
- moved K17,0 233.1 mm to (217.6, 27.8)
- moved K14,6 231.9 mm to (68.9, 189.0)
- moved D10,3 229.8 mm to (169.3, 200.9)
- moved K2,0 225.5 mm to (304.8, 108.4)
- moved K2,2 224.3 mm to (129.3, 168.9)
- moved K4,1 213.5 mm to (284.7, 88.3)
- moved K7,4 213.2 mm to (271.8, 48.0)
- moved K16,1 197.4 mm to (312.1, 48.0)
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
Commit message: Update KiCAD files
Parts:
- removed D14,66: D, keyboard_parts:D_SOD123_axial
- removed U999: TL750M05CKTTR, Package_TO_SOT_SMD:TO-263-3_TabPin2
- added D14,6: D, keyboard_parts:D_SOD123_axial, F.Cu at (419.4, 174.5)
- added U10: PCA9306D, Package_SO:SO-8_3.9x4.9mm_P1.27mm, F.Cu at (407.4, 211.6)
- added U11: TXB0104D, Package_SO:SOIC-14_3.9x8.7mm_P1.27mm, F.Cu at (410.5, 223.8)
- LD0,0, LD0,1, LD0,2, LD0,3, LD0,4, LD0,5, LD1,0, LD1,1, LD1,2, LD1,3, LD1,4, LD1,5, LD10,0, LD10,1, LD10,2, LD10,3, LD10,4, LD10,5, LD11,0, LD11,1, LD11,2, LD11,3, LD11,4, LD11,5, LD12,0, LD12,1, LD12,2, LD12,3, LD13,0, LD13,1, LD13,2, LD14,0, LD14,1, LD14,3, LD14,6, LD15,0, LD15,1, LD15,3, LD15,5, LD15,6, LD16,0, LD16,1, LD16,3, LD16,4, LD16,5, LD16,6, LD17,0, LD17,1, LD17,3, LD17,4, LD17,5, LD17,6, LD17,7, LD18,0, LD18,1, LD18,3, LD18,4, LD18,5, LD18,6, LD18,7, LD19,0, LD19,1, LD19,3, LD19,4, LD19,6, LD19,7, LD2,0, LD2,1, LD2,2, LD2,3, LD2,4, LD2,5, LD20,0, LD20,1, LD20,4, LD20,6, LD20,7, LD3,0, LD3,1, LD3,2, LD3,3, LD3,4, LD3,5, LD4,0, LD4,1, LD4,2, LD4,3, LD4,4, LD4,5, LD5,0, LD5,1, LD5,2, LD5,3, LD5,4, LD5,5, LD6,0, LD6,1, LD6,2, LD6,3, LD6,4, LD6,5, LD7,0, LD7,1, LD7,2, LD7,3, LD7,4, LD7,5, LD8,0, LD8,1, LD8,2, LD8,3, LD8,4, LD8,5, LD9,0, LD9,1, LD9,2, LD9,3, LD9,4, LD9,5: moved to B.Cu
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Connections:
- net Net-(K20,0-Pad1) renamed KEY_COL20
- D0,0 pad 1: Net-(D0,0-Pad1) -> KEY_ROW0
- D0,1 pad 1: Net-(D0,1-Pad1) -> KEY_ROW1
- D0,2 pad 1: Net-(D0,2-Pad1) -> KEY_ROW2
- D0,3 pad 1: Net-(D0,3-Pad1) -> KEY_ROW3
- D0,4 pad 1: Net-(D0,4-Pad1) -> KEY_ROW4
- D0,5 pad 1: Net-(D0,5-Pad1) -> KEY_ROW5
- D1,0 pad 1: Net-(D0,0-Pad1) -> KEY_ROW0
- D1,1 pad 1: Net-(D0,1-Pad1) -> KEY_ROW1
- D1,2 pad 1: Net-(D0,2-Pad1) -> KEY_ROW2
- D1,3 pad 1: Net-(D0,3-Pad1) -> KEY_ROW3
- D1,4 pad 1: Net-(D0,4-Pad1) -> KEY_ROW4
- D1,5 pad 1: Net-(D0,5-Pad1) -> KEY_ROW5
- D10,0 pad 1: Net-(D0,0-Pad1) -> KEY_ROW0
- D10,1 pad 1: Net-(D0,1-Pad1) -> KEY_ROW1
- D10,2 pad 1: Net-(D0,2-Pad1) -> KEY_ROW2
- D10,3 pad 1: Net-(D0,3-Pad1) -> KEY_ROW3
- D10,4 pad 1: Net-(D0,4-Pad1) -> KEY_ROW4
- D10,5 pad 1: Net-(D0,5-Pad1) -> KEY_ROW5
- D11,0 pad 1: Net-(D0,0-Pad1) -> KEY_ROW0
- D11,1 pad 1: Net-(D0,1-Pad1) -> KEY_ROW1
- D11,2 pad 1: Net-(D0,2-Pad1) -> KEY_ROW2
- D11,3 pad 1: Net-(D0,3-Pad1) -> KEY_ROW3
- D11,4 pad 1: Net-(D0,4-Pad1) -> KEY_ROW4
- D11,5 pad 1: Net-(D0,5-Pad1) -> KEY_ROW5
- D12,0 pad 1: Net-(D0,0-Pad1) -> KEY_ROW0
- D12,1 pad 1: Net-(D0,1-Pad1) -> KEY_ROW1
- D12,2 pad 1: Net-(D0,2-Pad1) -> KEY_ROW2
- D12,3 pad 1: Net-(D0,3-Pad1) -> KEY_ROW3
- D13,1 pad 1: Net-(D0,1-Pad1) -> KEY_ROW1
- D13,2 pad 1: Net-(D0,2-Pad1) -> KEY_ROW2
- D14,0 pad 1: Net-(D0,0-Pad1) -> KEY_ROW0
- D14,1 pad 1: Net-(D0,1-Pad1) -> KEY_ROW1
- D14,3 pad 1: Net-(D0,3-Pad1) -> KEY_ROW3
- D15,0 pad 1: Net-(D0,0-Pad1) -> KEY_ROW0
- D15,1 pad 1: Net-(D0,1-Pad1) -> KEY_ROW1
- D15,3 pad 1: Net-(D0,3-Pad1) -> KEY_ROW3
- D15,5 pad 1: Net-(D0,5-Pad1) -> KEY_ROW5
- D15,6 pad 1: Net-(D14,66-Pad1) -> KEY_ROW6
- D16,0 pad 1: Net-(D0,0-Pad1) -> KEY_ROW0
- D16,1 pad 1: Net-(D0,1-Pad1) -> KEY_ROW1
- D16,3 pad 1: Net-(D0,3-Pad1) -> KEY_ROW3
- D16,4 pad 1: Net-(D0,4-Pad1) -> KEY_ROW4
- D16,5 pad 1: Net-(D0,5-Pad1) -> KEY_ROW5
- D16,6 pad 1: Net-(D14,66-Pad1) -> KEY_ROW6
- D17,0 pad 1: Net-(D0,0-Pad1) -> KEY_ROW0
- D17,1 pad 1: Net-(D0,1-Pad1) -> KEY_ROW1
- D17,3 pad 1: Net-(D0,3-Pad1) -> KEY_ROW3
- D17,4 pad 1: Net-(D0,4-Pad1) -> KEY_ROW4
- D17,5 pad 1: Net-(D0,5-Pad1) -> KEY_ROW5
- D17,6 pad 1: Net-(D14,66-Pad1) -> KEY_ROW6
- D18,0 pad 1: Net-(D0,0-Pad1) -> KEY_ROW0
- D18,1 pad 1: Net-(D0,1-Pad1) -> KEY_ROW1
- D18,3 pad 1: Net-(D0,3-Pad1) -> KEY_ROW3
- D18,4 pad 1: Net-(D0,4-Pad1) -> KEY_ROW4
- D18,5 pad 1: Net-(D0,5-Pad1) -> KEY_ROW5
- D18,6 pad 1: Net-(D14,66-Pad1) -> KEY_ROW6
- D19,0 pad 1: Net-(D0,0-Pad1) -> KEY_ROW0
- D19,1 pad 1: Net-(D0,1-Pad1) -> KEY_ROW1
- D19,3 pad 1: Net-(D0,3-Pad1) -> KEY_ROW3
- D19,4 pad 1: Net-(D0,4-Pad1) -> KEY_ROW4
- D19,6 pad 1: Net-(D14,66-Pad1) -> KEY_ROW6
- D2,0 pad 1: Net-(D0,0-Pad1) -> KEY_ROW0
- D2,1 pad 1: Net-(D0,1-Pad1) -> KEY_ROW1
- D2,2 pad 1: Net-(D0,2-Pad1) -> KEY_ROW2
- D2,3 pad 1: Net-(D0,3-Pad1) -> KEY_ROW3
- D2,4 pad 1: Net-(D0,4-Pad1) -> KEY_ROW4
- D2,5 pad 1: Net-(D0,5-Pad1) -> KEY_ROW5
- D20,0 pad 1: Net-(D0,0-Pad1) -> KEY_ROW0
- D20,1 pad 1: Net-(D0,1-Pad1) -> KEY_ROW1
- D3,0 pad 1: Net-(D0,0-Pad1) -> KEY_ROW0
- D3,1 pad 1: Net-(D0,1-Pad1) -> KEY_ROW1
- D3,2 pad 1: Net-(D0,2-Pad1) -> KEY_ROW2
- D3,3 pad 1: Net-(D0,3-Pad1) -> KEY_ROW3
- D3,4 pad 1: Net-(D0,4-Pad1) -> KEY_ROW4
- D3,5 pad 1: Net-(D0,5-Pad1) -> KEY_ROW5
- D4,0 pad 1: Net-(D0,0-Pad1) -> KEY_ROW0
- D4,1 pad 1: Net-(D0,1-Pad1) -> KEY_ROW1
- D4,2 pad 1: Net-(D0,2-Pad1) -> KEY_ROW2
- D4,3 pad 1: Net-(D0,3-Pad1) -> KEY_ROW3
- D4,4 pad 1: Net-(D0,4-Pad1) -> KEY_ROW4
- D5,0 pad 1: Net-(D0,0-Pad1) -> KEY_ROW0
- D5,1 pad 1: Net-(D0,1-Pad1) -> KEY_ROW1
- D5,2 pad 1: Net-(D0,2-Pad1) -> KEY_ROW2
- D5,3 pad 1: Net-(D0,3-Pad1) -> KEY_ROW3
- D5,4 pad 1: Net-(D0,4-Pad1) -> KEY_ROW4
- D6,0 pad 1: Net-(D0,0-Pad1) -> KEY_ROW0
- D6,1 pad 1: Net-(D0,1-Pad1) -> KEY_ROW1
- D6,2 pad 1: Net-(D0,2-Pad1) -> KEY_ROW2
- D6,3 pad 1: Net-(D0,3-Pad1) -> KEY_ROW3
- D6,4 pad 1: Net-(D0,4-Pad1) -> KEY_ROW4
- D7,0 pad 1: Net-(D0,0-Pad1) -> KEY_ROW0
- D7,1 pad 1: Net-(D0,1-Pad1) -> KEY_ROW1
- D7,2 pad 1: Net-(D0,2-Pad1) -> KEY_ROW2
- D7,3 pad 1: Net-(D0,3-Pad1) -> KEY_ROW3
- D7,4 pad 1: Net-(D0,4-Pad1) -> KEY_ROW4
- D8,0 pad 1: Net-(D0,0-Pad1) -> KEY_ROW0
- D8,1 pad 1: Net-(D0,1-Pad1) -> KEY_ROW1
- D8,2 pad 1: Net-(D0,2-Pad1) -> KEY_ROW2
- D8,3 pad 1: Net-(D0,3-Pad1) -> KEY_ROW3
- D8,4 pad 1: Net-(D0,4-Pad1) -> KEY_ROW4
- D8,5 pad 1: Net-(D0,5-Pad1) -> KEY_ROW5
- D9,0 pad 1: Net-(D0,0-Pad1) -> KEY_ROW0
- D9,1 pad 1: Net-(D0,1-Pad1) -> KEY_ROW1
- D9,2 pad 1: Net-(D0,2-Pad1) -> KEY_ROW2
- D9,3 pad 1: Net-(D0,3-Pad1) -> KEY_ROW3
- D9,4 pad 1: Net-(D0,4-Pad1) -> KEY_ROW4
- D9,5 pad 1: Net-(D0,5-Pad1) -> KEY_ROW5
- J1 pad 1: I2C_SDA0 -> PICO_SDA0
- J1 pad 2: I2C_SCL0 -> PICO_SCL0
- K0,0 pad 1: Net-(K0,0-Pad1) -> KEY_COL0
- K0,1 pad 1: Net-(K0,0-Pad1) -> KEY_COL0
- K0,2 pad 1: Net-(K0,0-Pad1) -> KEY_COL0
- K0,3 pad 1: Net-(K0,0-Pad1) -> KEY_COL0
- K0,4 pad 1: Net-(K0,0-Pad1) -> KEY_COL0
- K0,5 pad 1: Net-(K0,0-Pad1) -> KEY_COL0
- K1,0 pad 1: Net-(K1,0-Pad1) -> KEY_COL1
- K1,1 pad 1: Net-(K1,0-Pad1) -> KEY_COL1
- K1,2 pad 1: Net-(K1,0-Pad1) -> KEY_COL1
- K1,3 pad 1: Net-(K1,0-Pad1) -> KEY_COL1
- K1,4 pad 1: Net-(K1,0-Pad1) -> KEY_COL1
- K1,5 pad 1: Net-(K1,0-Pad1) -> KEY_COL1
- K10,0 pad 1: Net-(K10,0-Pad1) -> KEY_COL10
- K10,1 pad 1: Net-(K10,0-Pad1) -> KEY_COL10
- K10,2 pad 1: Net-(K10,0-Pad1) -> KEY_COL10
- K10,3 pad 1: Net-(K10,0-Pad1) -> KEY_COL10
- K10,4 pad 1: Net-(K10,0-Pad1) -> KEY_COL10
- K10,5 pad 1: Net-(K10,0-Pad1) -> KEY_COL10
- K11,0 pad 1: Net-(K11,0-Pad1) -> KEY_COL11
- K11,1 pad 1: Net-(K11,0-Pad1) -> KEY_COL11
- K11,2 pad 1: Net-(K11,0-Pad1) -> KEY_COL11
- K11,3 pad 1: Net-(K11,0-Pad1) -> KEY_COL11
- K11,4 pad 1: Net-(K11,0-Pad1) -> KEY_COL11
- K11,5 pad 1: Net-(K11,0-Pad1) -> KEY_COL11
- K12,0 pad 1: Net-(K12,0-Pad1) -> KEY_COL12
- K12,1 pad 1: Net-(K12,0-Pad1) -> KEY_COL12
- K12,2 pad 1: Net-(K12,0-Pad1) -> KEY_COL12
- K12,3 pad 1: Net-(K12,0-Pad1) -> KEY_COL12
- K13,1 pad 1: Net-(K13,1-Pad1) -> KEY_COL13
- K13,2 pad 1: Net-(K13,1-Pad1) -> KEY_COL13
- K14,0 pad 1: Net-(K14,0-Pad1) -> KEY_COL14
- K14,1 pad 1: Net-(K14,0-Pad1) -> KEY_COL14
- K14,3 pad 1: Net-(K14,0-Pad1) -> KEY_COL14
- K14,6 pad 1: Net-(K14,0-Pad1) -> KEY_COL14
- K15,0 pad 1: Net-(K15,0-Pad1) -> KEY_COL15
- K15,1 pad 1: Net-(K15,0-Pad1) -> KEY_COL15
- K15,3 pad 1: Net-(K15,0-Pad1) -> KEY_COL15
- K15,5 pad 1: Net-(K15,0-Pad1) -> KEY_COL15
- K15,6 pad 1: Net-(K15,0-Pad1) -> KEY_COL15
- K16,0 pad 1: Net-(K16,0-Pad1) -> KEY_COL16
- K16,1 pad 1: Net-(K16,0-Pad1) -> KEY_COL16
- K16,3 pad 1: Net-(K16,0-Pad1) -> KEY_COL16
- K16,4 pad 1: Net-(K16,0-Pad1) -> KEY_COL16
- K16,5 pad 1: Net-(K16,0-Pad1) -> KEY_COL16
- K16,6 pad 1: Net-(K16,0-Pad1) -> KEY_COL16
- K17,0 pad 1: Net-(K17,0-Pad1) -> KEY_COL17
- K17,1 pad 1: Net-(K17,0-Pad1) -> KEY_COL17
- K17,3 pad 1: Net-(K17,0-Pad1) -> KEY_COL17
- K17,4 pad 1: Net-(K17,0-Pad1) -> KEY_COL17
- K17,5 pad 1: Net-(K17,0-Pad1) -> KEY_COL17
- K17,6 pad 1: Net-(K17,0-Pad1) -> KEY_COL17
- K18,0 pad 1: Net-(K18,0-Pad1) -> KEY_COL18
- K18,1 pad 1: Net-(K18,0-Pad1) -> KEY_COL18
- K18,3 pad 1: Net-(K18,0-Pad1) -> KEY_COL18
- K18,4 pad 1: Net-(K18,0-Pad1) -> KEY_COL18
- K18,5 pad 1: Net-(K18,0-Pad1) -> KEY_COL18
- K18,6 pad 1: Net-(K18,0-Pad1) -> KEY_COL18
- K19,0 pad 1: Net-(K19,0-Pad1) -> KEY_COL19
- K19,1 pad 1: Net-(K19,0-Pad1) -> KEY_COL19
- K19,3 pad 1: Net-(K19,0-Pad1) -> KEY_COL19
- K19,4 pad 1: Net-(K19,0-Pad1) -> KEY_COL19
- K19,6 pad 1: Net-(K19,0-Pad1) -> KEY_COL19
- K2,0 pad 1: Net-(K2,0-Pad1) -> KEY_COL2
- K2,1 pad 1: Net-(K2,0-Pad1) -> KEY_COL2
- K2,2 pad 1: Net-(K2,0-Pad1) -> KEY_COL2
- K2,3 pad 1: Net-(K2,0-Pad1) -> KEY_COL2
- K2,4 pad 1: Net-(K2,0-Pad1) -> KEY_COL2
- K2,5 pad 1: Net-(K2,0-Pad1) -> KEY_COL2
- K3,0 pad 1: Net-(K3,0-Pad1) -> KEY_COL3
- K3,1 pad 1: Net-(K3,0-Pad1) -> KEY_COL3
- K3,2 pad 1: Net-(K3,0-Pad1) -> KEY_COL3
- K3,3 pad 1: Net-(K3,0-Pad1) -> KEY_COL3
- K3,4 pad 1: Net-(K3,0-Pad1) -> KEY_COL3
- K3,5 pad 1: Net-(K3,0-Pad1) -> KEY_COL3
- K4,0 pad 1: Net-(K4,0-Pad1) -> KEY_COL4
- K4,1 pad 1: Net-(K4,0-Pad1) -> KEY_COL4
- K4,2 pad 1: Net-(K4,0-Pad1) -> KEY_COL4
- K4,3 pad 1: Net-(K4,0-Pad1) -> KEY_COL4
- K4,4 pad 1: Net-(K4,0-Pad1) -> KEY_COL4
- K5,0 pad 1: Net-(K5,0-Pad1) -> KEY_COL5
- K5,1 pad 1: Net-(K5,0-Pad1) -> KEY_COL5
- K5,2 pad 1: Net-(K5,0-Pad1) -> KEY_COL5
- K5,3 pad 1: Net-(K5,0-Pad1) -> KEY_COL5
- K5,4 pad 1: Net-(K5,0-Pad1) -> KEY_COL5
- K6,0 pad 1: Net-(K6,0-Pad1) -> KEY_COL6
- K6,1 pad 1: Net-(K6,0-Pad1) -> KEY_COL6
- K6,2 pad 1: Net-(K6,0-Pad1) -> KEY_COL6
- K6,3 pad 1: Net-(K6,0-Pad1) -> KEY_COL6
- K6,4 pad 1: Net-(K6,0-Pad1) -> KEY_COL6
- K7,0 pad 1: Net-(K7,0-Pad1) -> KEY_COL7
- K7,1 pad 1: Net-(K7,0-Pad1) -> KEY_COL7
- K7,2 pad 1: Net-(K7,0-Pad1) -> KEY_COL7
- K7,3 pad 1: Net-(K7,0-Pad1) -> KEY_COL7
- K7,4 pad 1: Net-(K7,0-Pad1) -> KEY_COL7
- K8,0 pad 1: Net-(K8,0-Pad1) -> KEY_COL8
- K8,1 pad 1: Net-(K8,0-Pad1) -> KEY_COL8
- K8,2 pad 1: Net-(K8,0-Pad1) -> KEY_COL8
- K8,3 pad 1: Net-(K8,0-Pad1) -> KEY_COL8
- K8,4 pad 1: Net-(K8,0-Pad1) -> KEY_COL8
- K8,5 pad 1: Net-(K8,0-Pad1) -> KEY_COL8
- K9,0 pad 1: Net-(K9,0-Pad1) -> KEY_COL9
- K9,1 pad 1: Net-(K9,0-Pad1) -> KEY_COL9
- K9,2 pad 1: Net-(K9,0-Pad1) -> KEY_COL9
- K9,3 pad 1: Net-(K9,0-Pad1) -> KEY_COL9
- K9,4 pad 1: Net-(K9,0-Pad1) -> KEY_COL9
- K9,5 pad 1: Net-(K9,0-Pad1) -> KEY_COL9
- LD0,0 pad 1: Net-(LD0,0-Pad1) -> MAIN_VBUS
- LD0,1 pad 1: Net-(LD0,0-Pad1) -> MAIN_VBUS
- LD0,2 pad 1: Net-(LD0,0-Pad1) -> MAIN_VBUS
- LD0,3 pad 1: Net-(LD0,0-Pad1) -> MAIN_VBUS
- LD0,4 pad 1: Net-(LD0,0-Pad1) -> MAIN_VBUS
- LD0,5 pad 1: Net-(LD0,0-Pad1) -> MAIN_VBUS
- LD1,0 pad 1: Net-(LD0,0-Pad1) -> MAIN_VBUS
- LD1,1 pad 1: Net-(LD0,0-Pad1) -> MAIN_VBUS
- LD1,2 pad 1: Net-(LD0,0-Pad1) -> MAIN_VBUS
- LD1,3 pad 1: Net-(LD0,0-Pad1) -> MAIN_VBUS
- LD1,4 pad 1: Net-(LD0,0-Pad1) -> MAIN_VBUS
- LD1,5 pad 1: Net-(LD0,0-Pad1) -> MAIN_VBUS
- LD10,0 pad 1: Net-(LD0,0-Pad1) -> MAIN_VBUS
- LD10,1 pad 1: Net-(LD0,0-Pad1) -> MAIN_VBUS
- LD10,2 pad 1: Net-(LD0,0-Pad1) -> MAIN_VBUS
- LD10,3 pad 1: Net-(LD0,0-Pad1) -> MAIN_VBUS
- LD10,4 pad 1: Net-(LD0,0-Pad1) -> MAIN_VBUS
- LD10,5 pad 1: Net-(LD0,0-Pad1) -> MAIN_VBUS
- LD11,0 pad 1: Net-(LD0,0-Pad1) -> MAIN_VBUS
- LD11,1 pad 1: Net-(LD0,0-Pad1) -> MAIN_VBUS
- LD11,2 pad 1: Net-(LD0,0-Pad1) -> MAIN_VBUS
- LD11,3 pad 1: Net-(LD0,0-Pad1) -> MAIN_VBUS
- LD11,4 pad 1: Net-(LD0,0-Pad1) -> MAIN_VBUS
- LD11,5 pad 1: Net-(LD0,0-Pad1) -> MAIN_VBUS
- LD12,0 pad 1: Net-(LD0,0-Pad1) -> MAIN_VBUS
- LD12,1 pad 1: Net-(LD0,0-Pad1) -> MAIN_VBUS
- LD12,2 pad 1: Net-(LD0,0-Pad1) -> MAIN_VBUS
- LD12,3 pad 1: Net-(LD0,0-Pad1) -> MAIN_VBUS
- LD13,0 pad 1: Net-(LD0,0-Pad1) -> MAIN_VBUS
- LD13,1 pad 1: Net-(LD0,0-Pad1) -> MAIN_VBUS
- LD13,2 pad 1: Net-(LD0,0-Pad1) -> MAIN_VBUS
- LD14,0 pad 1: Net-(LD0,0-Pad1) -> MAIN_VBUS
- LD14,1 pad 1: Net-(LD0,0-Pad1) -> MAIN_VBUS
- LD14,3 pad 1: Net-(LD0,0-Pad1) -> MAIN_VBUS
- LD14,6 pad 1: Net-(LD0,0-Pad1) -> MAIN_VBUS
- LD15,0 pad 1: Net-(LD0,0-Pad1) -> MAIN_VBUS
- LD15,1 pad 1: Net-(LD0,0-Pad1) -> MAIN_VBUS
- LD15,3 pad 1: Net-(LD0,0-Pad1) -> MAIN_VBUS
- LD15,5 pad 1: Net-(LD0,0-Pad1) -> MAIN_VBUS
- LD15,6 pad 1: Net-(LD0,0-Pad1) -> MAIN_VBUS
- LD16,0 pad 1: Net-(LD0,0-Pad1) -> MAIN_VBUS
- LD16,1 pad 1: Net-(LD0,0-Pad1) -> MAIN_VBUS
- LD16,3 pad 1: Net-(LD0,0-Pad1) -> MAIN_VBUS
- LD16,4 pad 1: Net-(LD0,0-Pad1) -> MAIN_VBUS
- LD16,5 pad 1: Net-(LD0,0-Pad1) -> MAIN_VBUS
- LD16,6 pad 1: Net-(LD0,0-Pad1) -> MAIN_VBUS
- LD17,0 pad 1: Net-(LD0,0-Pad1) -> MAIN_VBUS
- LD17,1 pad 1: Net-(LD0,0-Pad1) -> MAIN_VBUS
- LD17,3 pad 1: Net-(LD0,0-Pad1) -> MAIN_VBUS
- LD17,4 pad 1: Net-(LD0,0-Pad1) -> MAIN_VBUS
- LD17,5 pad 1: Net-(LD0,0-Pad1) -> MAIN_VBUS
- LD17,6 pad 1: Net-(LD0,0-Pad1) -> MAIN_VBUS
- LD17,7 pad 1: Net-(LD0,0-Pad1) -> MAIN_VBUS
- LD18,0 pad 1: Net-(LD0,0-Pad1) -> MAIN_VBUS
- LD18,1 pad 1: Net-(LD0,0-Pad1) -> MAIN_VBUS
- LD18,3 pad 1: Net-(LD0,0-Pad1) -> MAIN_VBUS
- LD18,4 pad 1: Net-(LD0,0-Pad1) -> MAIN_VBUS
- LD18,5 pad 1: Net-(LD0,0-Pad1) -> MAIN_VBUS
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Routing:
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Other:
- copper layers 2 -> 4
