File: KiCAD/RedPyKeeb.kicad_pcb (KiCad board)
At the start: 4 copper layers, 448.3 x 179.1 mm, 349 parts, among them J0 Conn_01x04, J1 Conn_01x04, J2 Conn_01x04, U1 MCP23017-E/SO, U10 PCA9306DP,118, U11 TXB0104D, U2 MCP23017-E/SO, U3 MCP23017-E/SO

Commit message: KiCAD and firmware updates, first working firmware and half way through a board rewire after the initial semi-working board. Firmware has no real LED control other than the power budget system and pin setup. Although the firmware works, it is not a working keyboard, yet.
Parts:
- removed C3: 0805B104K100CT, Capacitors_SMD:C_0805_HandSoldering
- removed U3: MCP23017-E/SO, Package_SO:SOIC-28W_7.5x17.9mm_P1.27mm
- added LD3,5,0: APA102 2020, Custom_pico:LED-APA102-2020, F.Cu at (177.1, 199.4)
- added LD3,5,1: APA102 2020, Custom_pico:LED-APA102-2020, F.Cu at (241.2, 199.3)
- moved C6 5.46 mm to (492.4, 78.3)
- moved J2 5.46 mm to (446.0, 56.3)
- moved R2 5.46 mm to (461.1, 87.2)
- moved U10 5.46 mm to (456.3, 84.7)
- moved C5 5.46 mm to (439.0, 85.6)
- moved C7 5.46 mm to (439.1, 80.4)
- moved J1 5.46 mm to (481.7, 86.0)
- moved R1 5.46 mm to (459.1, 87.2)
- moved U0 5.46 mm to (432.9, 72.5)
- moved U11 5.46 mm to (444.8, 84.1)
- moved J0 5.46 mm to (487.9, 65.8)
- moved C4 5.46 mm to (453.5, 87.9)
- moved R3 5.46 mm to (461.2, 83.9)
- moved R4 5.46 mm to (459.4, 79.3)
- moved R5 5.46 mm to (457.5, 79.3)
Connections:
- net PICO_RUN renamed Net-(U0-Pad30)
- LD0,1 pad 4: LED_SDA_ROW1 -> Net-(LD0,1-Pad4)
- LD0,1 pad 5: LED_SCL_ROW1 -> Net-(LD0,1-Pad5)
- LD0,2 pad 4: LED_SDA_ROW2 -> Net-(LD0,2-Pad4)
- LD0,2 pad 5: LED_SCL_ROW2 -> Net-(LD0,2-Pad5)
- LD0,3 pad 4: LED_SDA_ROW3 -> Net-(LD0,3-Pad4)
- LD0,3 pad 5: LED_SCL_ROW3 -> Net-(LD0,3-Pad5)
- LD0,4 pad 4: LED_SDA_ROW4 -> Net-(LD0,3-Pad3)
- LD0,4 pad 5: LED_SCL_ROW4 -> Net-(LD0,3-Pad2)
- LD0,5 pad 4: LED_SDA_ROW5 -> Net-(LD0,5-Pad4)
- LD0,5 pad 5: LED_SCL_ROW5 -> Net-(LD0,5-Pad5)
- LD1,3 pad 2: Net-(LD1,3-Pad2) -> Net-(LD0,3-Pad5)
- LD1,3 pad 3: Net-(LD1,3-Pad3) -> Net-(LD0,3-Pad4)
- LD1,3 pad 4: Net-(LD0,3-Pad3) -> Net-(LD1,3-Pad4)
- LD1,3 pad 5: Net-(LD0,3-Pad2) -> Net-(LD1,3-Pad5)
- LD1,5 pad 2: Net-(LD1,5-Pad2) -> Net-(LD0,5-Pad5)
- LD1,5 pad 3: Net-(LD1,5-Pad3) -> Net-(LD0,5-Pad4)
- LD1,5 pad 4: Net-(LD0,5-Pad3) -> Net-(LD1,5-Pad4)
- LD1,5 pad 5: Net-(LD0,5-Pad2) -> Net-(LD1,5-Pad5)
- LD11,3 pad 2: Net-(LD11,3-Pad2) -> Net-(LD10,3-Pad5)
- LD11,3 pad 3: Net-(LD11,3-Pad3) -> Net-(LD10,3-Pad4)
- LD11,3 pad 4: Net-(LD10,3-Pad3) -> Net-(LD11,3-Pad4)
- LD11,3 pad 5: Net-(LD10,3-Pad2) -> Net-(LD11,3-Pad5)
- LD11,5 pad 2: Net-(LD11,5-Pad2) -> Net-(LD10,5-Pad5)
- LD11,5 pad 3: Net-(LD11,5-Pad3) -> Net-(LD10,5-Pad4)
- LD11,5 pad 4: Net-(LD10,5-Pad3) -> Net-(LD11,5-Pad4)
- LD11,5 pad 5: Net-(LD10,5-Pad2) -> Net-(LD11,5-Pad5)
- LD12,3 pad 2: Net-(LD12,3-Pad2) -> Net-(LD11,3-Pad5)
- LD12,3 pad 3: Net-(LD12,3-Pad3) -> Net-(LD11,3-Pad4)
- LD12,3 pad 4: Net-(LD11,3-Pad3) -> Net-(LD12,3-Pad4)
- LD12,3 pad 5: Net-(LD11,3-Pad2) -> Net-(LD12,3-Pad5)
- LD14,3 pad 2: Net-(LD14,3-Pad2) -> Net-(LD12,3-Pad5)
- LD14,3 pad 3: Net-(LD14,3-Pad3) -> Net-(LD12,3-Pad4)
- LD14,3 pad 4: Net-(LD12,3-Pad3) -> Net-(LD14,3-Pad4)
- LD14,3 pad 5: Net-(LD12,3-Pad2) -> Net-(LD14,3-Pad5)
- LD14,6 pad 4: LED_SDA_ROW6 -> Net-(LD0,5-Pad3)
- LD14,6 pad 5: LED_SCL_ROW6 -> Net-(LD0,5-Pad2)
- LD15,3 pad 2: Net-(LD15,3-Pad2) -> Net-(LD14,3-Pad5)
- LD15,3 pad 3: Net-(LD15,3-Pad3) -> Net-(LD14,3-Pad4)
- LD15,3 pad 4: Net-(LD14,3-Pad3) -> Net-(LD15,3-Pad4)
- LD15,3 pad 5: Net-(LD14,3-Pad2) -> Net-(LD15,3-Pad5)
- LD15,5 pad 2: Net-(LD15,5-Pad2) -> Net-(LD11,5-Pad5)
- LD15,5 pad 3: Net-(LD15,5-Pad3) -> Net-(LD11,5-Pad4)
- LD15,5 pad 4: Net-(LD11,5-Pad3) -> Net-(LD15,5-Pad4)
- LD15,5 pad 5: Net-(LD11,5-Pad2) -> Net-(LD15,5-Pad5)
- LD16,3 pad 2: Net-(LD16,3-Pad2) -> Net-(LD15,3-Pad5)
- LD16,3 pad 3: Net-(LD16,3-Pad3) -> Net-(LD15,3-Pad4)
- LD16,3 pad 4: Net-(LD15,3-Pad3) -> Net-(LD16,3-Pad4)
- LD16,3 pad 5: Net-(LD15,3-Pad2) -> Net-(LD16,3-Pad5)
- LD16,5 pad 2: Net-(LD16,5-Pad2) -> Net-(LD15,5-Pad5)
- LD16,5 pad 3: Net-(LD16,5-Pad3) -> Net-(LD15,5-Pad4)
- LD16,5 pad 4: Net-(LD15,5-Pad3) -> Net-(LD16,5-Pad4)
- LD16,5 pad 5: Net-(LD15,5-Pad2) -> Net-(LD16,5-Pad5)
- LD17,3 pad 2: Net-(LD17,3-Pad2) -> Net-(LD16,3-Pad5)
- LD17,3 pad 3: Net-(LD17,3-Pad3) -> Net-(LD16,3-Pad4)
- LD17,3 pad 4: Net-(LD16,3-Pad3) -> Net-(LD17,3-Pad4)
- LD17,3 pad 5: Net-(LD16,3-Pad2) -> Net-(LD17,3-Pad5)
- LD17,5 pad 2: Net-(LD17,5-Pad2) -> Net-(LD16,5-Pad5)
- LD17,5 pad 3: Net-(LD17,5-Pad3) -> Net-(LD16,5-Pad4)
- LD17,5 pad 4: Net-(LD16,5-Pad3) -> Net-(LD17,5-Pad4)
- LD17,5 pad 5: Net-(LD16,5-Pad2) -> Net-(LD17,5-Pad5)
- LD17,7 pad 4: LED_SDA_ROW7 -> LED_SDA_STATUS0
- LD17,7 pad 5: LED_SCL_ROW7 -> LED_SCL_STATUS0
- LD18,3 pad 2: Net-(LD18,3-Pad2) -> Net-(LD17,3-Pad5)
- LD18,3 pad 3: Net-(LD18,3-Pad3) -> Net-(LD17,3-Pad4)
- LD18,3 pad 4: Net-(LD17,3-Pad3) -> Net-(LD18,3-Pad4)
- LD18,3 pad 5: Net-(LD17,3-Pad2) -> Net-(LD18,3-Pad5)
- LD18,5 pad 2: Net-(LD18,5-Pad2) -> Net-(LD17,5-Pad5)
- LD18,5 pad 3: Net-(LD18,5-Pad3) -> Net-(LD17,5-Pad4)
- LD18,5 pad 4: Net-(LD17,5-Pad3) -> Net-(LD18,5-Pad4)
- LD18,5 pad 5: Net-(LD17,5-Pad2) -> Net-(LD18,5-Pad5)
- LD19,3 pad 2: Net-(LD19,3-Pad2) -> Net-(LD18,3-Pad5)
- LD19,3 pad 3: Net-(LD19,3-Pad3) -> Net-(LD18,3-Pad4)
- LD19,3 pad 4: Net-(LD18,3-Pad3) -> Net-(LD13,2-Pad3)
- LD19,3 pad 5: Net-(LD18,3-Pad2) -> Net-(LD13,2-Pad2)
- LD19,4 pad 2: Net-(LD19,4-Pad2) -> Net-(LD18,5-Pad5)
- LD19,4 pad 3: Net-(LD19,4-Pad3) -> Net-(LD18,5-Pad4)
- LD2,3 pad 2: Net-(LD2,3-Pad2) -> Net-(LD1,3-Pad5)
- LD2,3 pad 3: Net-(LD2,3-Pad3) -> Net-(LD1,3-Pad4)
- LD2,3 pad 4: Net-(LD1,3-Pad3) -> Net-(LD2,3-Pad4)
- LD2,3 pad 5: Net-(LD1,3-Pad2) -> Net-(LD2,3-Pad5)
- LD2,5 pad 2: Net-(LD2,5-Pad2) -> Net-(LD1,5-Pad5)
- LD2,5 pad 3: Net-(LD2,5-Pad3) -> Net-(LD1,5-Pad4)
- LD2,5 pad 4: Net-(LD1,5-Pad3) -> Net-(LD2,5-Pad4)
- LD2,5 pad 5: Net-(LD1,5-Pad2) -> Net-(LD2,5-Pad5)
- LD20,0 pad 2: Net-(LD20,0-Pad2) -> Net-(LD0,1-Pad5)
- LD20,0 pad 3: Net-(LD20,0-Pad3) -> Net-(LD0,1-Pad4)
- LD20,1 pad 2: Net-(LD20,1-Pad2) -> Net-(LD0,2-Pad5)
- LD20,1 pad 3: Net-(LD20,1-Pad3) -> Net-(LD0,2-Pad4)
- LD3,3 pad 2: Net-(LD3,3-Pad2) -> Net-(LD2,3-Pad5)
- LD3,3 pad 3: Net-(LD3,3-Pad3) -> Net-(LD2,3-Pad4)
- LD3,3 pad 4: Net-(LD2,3-Pad3) -> Net-(LD3,3-Pad4)
- LD3,3 pad 5: Net-(LD2,3-Pad2) -> Net-(LD3,3-Pad5)
- LD3,5 pad 2: Net-(LD3,5-Pad2) -> Net-(LD3,5,0-Pad5)
- LD3,5 pad 3: Net-(LD3,5-Pad3) -> Net-(LD3,5,0-Pad4)
- LD3,5 pad 4: Net-(LD2,5-Pad3) -> Net-(LD3,5,1-Pad3)
- LD3,5 pad 5: Net-(LD2,5-Pad2) -> Net-(LD3,5,1-Pad2)
- LD4,3 pad 2: Net-(LD4,3-Pad2) -> Net-(LD3,3-Pad5)
- LD4,3 pad 3: Net-(LD4,3-Pad3) -> Net-(LD3,3-Pad4)
- LD4,3 pad 4: Net-(LD3,3-Pad3) -> Net-(LD4,3-Pad4)
- LD4,3 pad 5: Net-(LD3,3-Pad2) -> Net-(LD4,3-Pad5)
- LD5,3 pad 2: Net-(LD5,3-Pad2) -> Net-(LD4,3-Pad5)
- LD5,3 pad 3: Net-(LD5,3-Pad3) -> Net-(LD4,3-Pad4)
- LD5,3 pad 4: Net-(LD4,3-Pad3) -> Net-(LD5,3-Pad4)
- LD5,3 pad 5: Net-(LD4,3-Pad2) -> Net-(LD5,3-Pad5)
- LD6,3 pad 2: Net-(LD6,3-Pad2) -> Net-(LD5,3-Pad5)
- LD6,3 pad 3: Net-(LD6,3-Pad3) -> Net-(LD5,3-Pad4)
- LD6,3 pad 4: Net-(LD5,3-Pad3) -> Net-(LD6,3-Pad4)
- LD6,3 pad 5: Net-(LD5,3-Pad2) -> Net-(LD6,3-Pad5)
- LD7,3 pad 2: Net-(LD7,3-Pad2) -> Net-(LD6,3-Pad5)
- LD7,3 pad 3: Net-(LD7,3-Pad3) -> Net-(LD6,3-Pad4)
- LD7,3 pad 4: Net-(LD6,3-Pad3) -> Net-(LD7,3-Pad4)
- LD7,3 pad 5: Net-(LD6,3-Pad2) -> Net-(LD7,3-Pad5)
- LD8,3 pad 2: Net-(LD8,3-Pad2) -> Net-(LD7,3-Pad5)
- LD8,3 pad 3: Net-(LD8,3-Pad3) -> Net-(LD7,3-Pad4)
- LD8,3 pad 4: Net-(LD7,3-Pad3) -> Net-(LD8,3-Pad4)
- LD8,3 pad 5: Net-(LD7,3-Pad2) -> Net-(LD8,3-Pad5)
- LD8,5 pad 2: Net-(LD8,5-Pad2) -> Net-(LD3,5,1-Pad5)
- LD8,5 pad 3: Net-(LD8,5-Pad3) -> Net-(LD3,5,1-Pad4)
- LD8,5 pad 4: Net-(LD3,5-Pad3) -> Net-(LD8,5-Pad4)
- LD8,5 pad 5: Net-(LD3,5-Pad2) -> Net-(LD8,5-Pad5)
- LD9,3 pad 2: Net-(LD10,3-Pad5) -> Net-(LD8,3-Pad5)
- LD9,3 pad 3: Net-(LD10,3-Pad4) -> Net-(LD8,3-Pad4)
- LD9,3 pad 4: Net-(LD8,3-Pad3) -> Net-(LD10,3-Pad3)
- LD9,3 pad 5: Net-(LD8,3-Pad2) -> Net-(LD10,3-Pad2)
- LD9,5 pad 2: Net-(LD10,5-Pad5) -> Net-(LD8,5-Pad5)
- LD9,5 pad 3: Net-(LD10,5-Pad4) -> Net-(LD8,5-Pad4)
- LD9,5 pad 4: Net-(LD8,5-Pad3) -> Net-(LD10,5-Pad3)
- LD9,5 pad 5: Net-(LD8,5-Pad2) -> Net-(LD10,5-Pad2)
- U0 pad 14: Net-(U0-Pad14) -> LED_SCL_STATUS0
- U0 pad 15: Net-(U0-Pad15) -> LED_SDA_STATUS0
- U0 pad 19: Net-(U0-Pad19) -> LED_SCL_ROW0
- U0 pad 20: Net-(U0-Pad20) -> LED_SDA_ROW0
Routing:
- net GNDPWR: track 3543.4 -> 745.8 mm, vias 9 -> 2
- net Net-(LD0,1-Pad5): track 0.00 -> 449.6 mm
- net Net-(LD0,1-Pad4): track 0.00 -> 439.4 mm
- net LED_SCL_ROW6: track 402.6 -> 0.00 mm, vias 2 -> 0
- net LED_SCL_ROW7: track 381.1 -> 0.00 mm, vias 2 -> 0
- net LED_SDA_ROW7: track 379.2 -> 0.00 mm, vias 2 -> 0
- net LED_SDA_ROW6: track 378.2 -> 0.00 mm, vias 2 -> 0
- net LED_SDA_ROW0: track 6.70 -> 370.1 mm, vias 0 -> 2
- net LED_SCL_ROW0: track 11.0 -> 372.4 mm, vias 2 -> 0
- net PICO_33_REF: track 497.6 -> 138.1 mm, vias 3 -> 2
- net LED_SCL_STATUS0: track 0.00 -> 168.3 mm, vias 0 -> 2
- net LED_SDA_STATUS0: track 0.00 -> 167.6 mm
- net LED_SDA_ROW5: track 146.5 -> 0.00 mm, vias 2 -> 0
- net LED_SCL_ROW5: track 144.5 -> 0.00 mm, vias 2 -> 0
- net LED_SDA_ROW4: track 144.0 -> 0.00 mm, vias 2 -> 0
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
Commit message: Update KiCAD and firmware files. Firmware has had a little bit of work to make sending key data easier. PCB has been fully routed for the 4th time and should be good to test LEDs and a much more populated board.
Parts:
- D0,0, D0,1, D0,2, D0,3, D0,4, D0,5, D1,0, D1,1, D1,2, D1,3, D1,4, D1,5, D10,0, D10,1, D10,2, D10,3, D10,4, D10,5, D11,0, D11,1, D11,2, D11,3, D11,4, D11,5, D12,0, D12,1, D12,2, D12,3, D13,1, D13,2, D14,0, D14,1, D14,3, D14,6, D15,0, D15,1, D15,3, D15,5, D15,6, D16,0, D16,1, D16,3, D16,4, D16,5, D16,6, D17,0, D17,1, D17,3, D17,4, D17,5, D17,6, D18,0, D18,1, D18,3, D18,4, D18,5, D18,6, D19,0, D19,1, D19,3, D19,4, D19,6, D2,0, D2,1, D2,2, D2,3, D2,4, D2,5, D20,0, D20,1, D3,0, D3,1, D3,2, D3,3, D3,4, D3,5, D4,0, D4,1, D4,2, D4,3, D4,4, D5,0, D5,1, D5,2, D5,3, D5,4, D6,0, D6,1, D6,2, D6,3, D6,4, D7,0, D7,1, D7,2, D7,3, D7,4, D8,0, D8,1, D8,2, D8,3, D8,4, D8,5, D9,0, D9,1, D9,2, D9,3, D9,4, D9,5: value BAT54W-HG3-08 -> 1N4148W-7-F
- moved D10,0 1.48 mm to (312.0, 103.7)
- moved D12,0 1.48 mm to (350.6, 103.7)
- moved K11,0 1.48 mm to (339.2, 102.5)
- moved K8,0 1.48 mm to (274.1, 102.5)
- moved K9,0 1.48 mm to (300.5, 102.5)
- moved LD11,0 1.48 mm to (339.3, 95.5)
- moved LD8,0 1.48 mm to (274.3, 95.5)
- moved LD9,0 1.48 mm to (300.7, 95.5)
- moved D1,0 1.48 mm to (119.0, 103.8)
- moved D2,0 1.48 mm to (138.3, 103.7)
- moved D3,0 1.48 mm to (157.6, 103.7)
- moved D4,0 1.48 mm to (176.9, 103.7)
- moved D5,0 1.48 mm to (208.4, 103.7)
- moved D6,0 1.48 mm to (227.7, 103.7)
- moved D7,0 1.48 mm to (247.0, 103.7)
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Connections:
- LD0,4 pad 4: Net-(LD0,3-Pad3) -> Net-(LD0,4-Pad4)
- LD0,4 pad 5: Net-(LD0,3-Pad2) -> Net-(LD0,4-Pad5)
- LD1,3 pad 2: Net-(LD0,3-Pad5) -> Net-(LD1,3-Pad2)
- LD1,3 pad 3: Net-(LD0,3-Pad4) -> Net-(LD1,3-Pad3)
- LD1,3 pad 4: Net-(LD1,3-Pad4) -> Net-(LD0,3-Pad3)
- LD1,3 pad 5: Net-(LD1,3-Pad5) -> Net-(LD0,3-Pad2)
- LD1,5 pad 2: Net-(LD0,5-Pad5) -> Net-(LD1,5-Pad2)
- LD1,5 pad 3: Net-(LD0,5-Pad4) -> Net-(LD1,5-Pad3)
- LD1,5 pad 4: Net-(LD1,5-Pad4) -> Net-(LD0,5-Pad3)
- LD1,5 pad 5: Net-(LD1,5-Pad5) -> Net-(LD0,5-Pad2)
- LD11,3 pad 2: Net-(LD10,3-Pad5) -> Net-(LD11,3-Pad2)
- LD11,3 pad 3: Net-(LD10,3-Pad4) -> Net-(LD11,3-Pad3)
- LD11,3 pad 4: Net-(LD11,3-Pad4) -> Net-(LD10,3-Pad3)
- LD11,3 pad 5: Net-(LD11,3-Pad5) -> Net-(LD10,3-Pad2)
- LD11,5 pad 2: Net-(LD10,5-Pad5) -> Net-(LD11,5-Pad2)
- LD11,5 pad 3: Net-(LD10,5-Pad4) -> Net-(LD11,5-Pad3)
- LD11,5 pad 4: Net-(LD11,5-Pad4) -> Net-(LD10,5-Pad3)
- LD11,5 pad 5: Net-(LD11,5-Pad5) -> Net-(LD10,5-Pad2)
- LD12,3 pad 2: Net-(LD11,3-Pad5) -> Net-(LD12,3-Pad2)
- LD12,3 pad 3: Net-(LD11,3-Pad4) -> Net-(LD12,3-Pad3)
- LD12,3 pad 4: Net-(LD12,3-Pad4) -> Net-(LD11,3-Pad3)
- LD12,3 pad 5: Net-(LD12,3-Pad5) -> Net-(LD11,3-Pad2)
- LD13,2 pad 2: Net-(LD13,2-Pad2) -> Net-(LD0,3-Pad5)
- LD13,2 pad 3: Net-(LD13,2-Pad3) -> Net-(LD0,3-Pad4)
- LD14,3 pad 2: Net-(LD12,3-Pad5) -> Net-(LD14,3-Pad2)
- LD14,3 pad 3: Net-(LD12,3-Pad4) -> Net-(LD14,3-Pad3)
- LD14,3 pad 4: Net-(LD14,3-Pad4) -> Net-(LD12,3-Pad3)
- LD14,3 pad 5: Net-(LD14,3-Pad5) -> Net-(LD12,3-Pad2)
- LD14,6 pad 4: Net-(LD0,5-Pad3) -> Net-(LD14,6-Pad4)
- LD14,6 pad 5: Net-(LD0,5-Pad2) -> Net-(LD14,6-Pad5)
- LD15,3 pad 2: Net-(LD14,3-Pad5) -> Net-(LD15,3-Pad2)
- LD15,3 pad 3: Net-(LD14,3-Pad4) -> Net-(LD15,3-Pad3)
- LD15,3 pad 4: Net-(LD15,3-Pad4) -> Net-(LD14,3-Pad3)
- LD15,3 pad 5: Net-(LD15,3-Pad5) -> Net-(LD14,3-Pad2)
- LD15,5 pad 2: Net-(LD11,5-Pad5) -> Net-(LD15,5-Pad2)
- LD15,5 pad 3: Net-(LD11,5-Pad4) -> Net-(LD15,5-Pad3)
- LD15,5 pad 4: Net-(LD15,5-Pad4) -> Net-(LD11,5-Pad3)
- LD15,5 pad 5: Net-(LD15,5-Pad5) -> Net-(LD11,5-Pad2)
- LD16,3 pad 2: Net-(LD15,3-Pad5) -> Net-(LD16,3-Pad2)
- LD16,3 pad 3: Net-(LD15,3-Pad4) -> Net-(LD16,3-Pad3)
- LD16,3 pad 4: Net-(LD16,3-Pad4) -> Net-(LD15,3-Pad3)
- LD16,3 pad 5: Net-(LD16,3-Pad5) -> Net-(LD15,3-Pad2)
- LD16,5 pad 2: Net-(LD15,5-Pad5) -> Net-(LD16,5-Pad2)
- LD16,5 pad 3: Net-(LD15,5-Pad4) -> Net-(LD16,5-Pad3)
- LD16,5 pad 4: Net-(LD16,5-Pad4) -> Net-(LD15,5-Pad3)
- LD16,5 pad 5: Net-(LD16,5-Pad5) -> Net-(LD15,5-Pad2)
- LD17,3 pad 2: Net-(LD16,3-Pad5) -> Net-(LD17,3-Pad2)
- LD17,3 pad 3: Net-(LD16,3-Pad4) -> Net-(LD17,3-Pad3)
- LD17,3 pad 4: Net-(LD17,3-Pad4) -> Net-(LD16,3-Pad3)
- LD17,3 pad 5: Net-(LD17,3-Pad5) -> Net-(LD16,3-Pad2)
- LD17,5 pad 2: Net-(LD16,5-Pad5) -> Net-(LD17,5-Pad2)
- LD17,5 pad 3: Net-(LD16,5-Pad4) -> Net-(LD17,5-Pad3)
- LD17,5 pad 4: Net-(LD17,5-Pad4) -> Net-(LD16,5-Pad3)
- LD17,5 pad 5: Net-(LD17,5-Pad5) -> Net-(LD16,5-Pad2)
- LD18,3 pad 2: Net-(LD17,3-Pad5) -> Net-(LD18,3-Pad2)
- LD18,3 pad 3: Net-(LD17,3-Pad4) -> Net-(LD18,3-Pad3)
- LD18,3 pad 4: Net-(LD18,3-Pad4) -> Net-(LD17,3-Pad3)
- LD18,3 pad 5: Net-(LD18,3-Pad5) -> Net-(LD17,3-Pad2)
- LD18,5 pad 2: Net-(LD17,5-Pad5) -> Net-(LD14,6-Pad5)
- LD18,5 pad 3: Net-(LD17,5-Pad4) -> Net-(LD14,6-Pad4)
- LD18,5 pad 4: Net-(LD18,5-Pad4) -> Net-(LD17,5-Pad3)
- LD18,5 pad 5: Net-(LD18,5-Pad5) -> Net-(LD17,5-Pad2)
- LD19,3 pad 2: Net-(LD18,3-Pad5) -> Net-(LD0,4-Pad5)
- LD19,3 pad 3: Net-(LD18,3-Pad4) -> Net-(LD0,4-Pad4)
- LD19,3 pad 4: Net-(LD13,2-Pad3) -> Net-(LD18,3-Pad3)
- LD19,3 pad 5: Net-(LD13,2-Pad2) -> Net-(LD18,3-Pad2)
- LD19,4 pad 2: Net-(LD18,5-Pad5) -> Net-(LD0,5-Pad5)
- LD19,4 pad 3: Net-(LD18,5-Pad4) -> Net-(LD0,5-Pad4)
- LD2,3 pad 2: Net-(LD1,3-Pad5) -> Net-(LD2,3-Pad2)
- LD2,3 pad 3: Net-(LD1,3-Pad4) -> Net-(LD2,3-Pad3)
- LD2,3 pad 4: Net-(LD2,3-Pad4) -> Net-(LD1,3-Pad3)
- LD2,3 pad 5: Net-(LD2,3-Pad5) -> Net-(LD1,3-Pad2)
- LD2,5 pad 2: Net-(LD1,5-Pad5) -> Net-(LD2,5-Pad2)
- LD2,5 pad 3: Net-(LD1,5-Pad4) -> Net-(LD2,5-Pad3)
- LD2,5 pad 4: Net-(LD2,5-Pad4) -> Net-(LD1,5-Pad3)
- LD2,5 pad 5: Net-(LD2,5-Pad5) -> Net-(LD1,5-Pad2)
- LD3,3 pad 2: Net-(LD2,3-Pad5) -> Net-(LD3,3-Pad2)
- LD3,3 pad 3: Net-(LD2,3-Pad4) -> Net-(LD3,3-Pad3)
- LD3,3 pad 4: Net-(LD3,3-Pad4) -> Net-(LD2,3-Pad3)
- LD3,3 pad 5: Net-(LD3,3-Pad5) -> Net-(LD2,3-Pad2)
- LD3,5 pad 2: Net-(LD3,5,0-Pad5) -> Net-(LD3,5,1-Pad5)
- LD3,5 pad 3: Net-(LD3,5,0-Pad4) -> Net-(LD3,5,1-Pad4)
- LD3,5 pad 4: Net-(LD3,5,1-Pad3) -> Net-(LD3,5,0-Pad3)
- LD3,5 pad 5: Net-(LD3,5,1-Pad2) -> Net-(LD3,5,0-Pad2)
- LD3,5,0 pad 2: Net-(LD2,5-Pad5) -> Net-(LD3,5,0-Pad2)
- LD3,5,0 pad 3: Net-(LD2,5-Pad4) -> Net-(LD3,5,0-Pad3)
- LD3,5,0 pad 4: Net-(LD3,5,0-Pad4) -> Net-(LD2,5-Pad3)
- LD3,5,0 pad 5: Net-(LD3,5,0-Pad5) -> Net-(LD2,5-Pad2)
- LD4,3 pad 2: Net-(LD3,3-Pad5) -> Net-(LD4,3-Pad2)
- LD4,3 pad 3: Net-(LD3,3-Pad4) -> Net-(LD4,3-Pad3)
- LD4,3 pad 4: Net-(LD4,3-Pad4) -> Net-(LD3,3-Pad3)
- LD4,3 pad 5: Net-(LD4,3-Pad5) -> Net-(LD3,3-Pad2)
- LD5,3 pad 2: Net-(LD4,3-Pad5) -> Net-(LD5,3-Pad2)
- LD5,3 pad 3: Net-(LD4,3-Pad4) -> Net-(LD5,3-Pad3)
- LD5,3 pad 4: Net-(LD5,3-Pad4) -> Net-(LD4,3-Pad3)
- LD5,3 pad 5: Net-(LD5,3-Pad5) -> Net-(LD4,3-Pad2)
- LD6,3 pad 2: Net-(LD5,3-Pad5) -> Net-(LD6,3-Pad2)
- LD6,3 pad 3: Net-(LD5,3-Pad4) -> Net-(LD6,3-Pad3)
- LD6,3 pad 4: Net-(LD6,3-Pad4) -> Net-(LD5,3-Pad3)
- LD6,3 pad 5: Net-(LD6,3-Pad5) -> Net-(LD5,3-Pad2)
- LD7,3 pad 2: Net-(LD6,3-Pad5) -> Net-(LD7,3-Pad2)
- LD7,3 pad 3: Net-(LD6,3-Pad4) -> Net-(LD7,3-Pad3)
- LD7,3 pad 4: Net-(LD7,3-Pad4) -> Net-(LD6,3-Pad3)
- LD7,3 pad 5: Net-(LD7,3-Pad5) -> Net-(LD6,3-Pad2)
- LD8,3 pad 2: Net-(LD7,3-Pad5) -> Net-(LD8,3-Pad2)
- LD8,3 pad 3: Net-(LD7,3-Pad4) -> Net-(LD8,3-Pad3)
- LD8,3 pad 4: Net-(LD8,3-Pad4) -> Net-(LD7,3-Pad3)
- LD8,3 pad 5: Net-(LD8,3-Pad5) -> Net-(LD7,3-Pad2)
- LD8,5 pad 2: Net-(LD3,5,1-Pad5) -> Net-(LD8,5-Pad2)
- LD8,5 pad 3: Net-(LD3,5,1-Pad4) -> Net-(LD8,5-Pad3)
- LD8,5 pad 4: Net-(LD8,5-Pad4) -> Net-(LD3,5,1-Pad3)
- LD8,5 pad 5: Net-(LD8,5-Pad5) -> Net-(LD3,5,1-Pad2)
- LD9,3 pad 2: Net-(LD8,3-Pad5) -> Net-(LD10,3-Pad5)
- LD9,3 pad 3: Net-(LD8,3-Pad4) -> Net-(LD10,3-Pad4)
- LD9,3 pad 4: Net-(LD10,3-Pad3) -> Net-(LD8,3-Pad3)
- LD9,3 pad 5: Net-(LD10,3-Pad2) -> Net-(LD8,3-Pad2)
- LD9,5 pad 2: Net-(LD8,5-Pad5) -> Net-(LD10,5-Pad5)
- LD9,5 pad 3: Net-(LD8,5-Pad4) -> Net-(LD10,5-Pad4)
- LD9,5 pad 4: Net-(LD10,5-Pad3) -> Net-(LD8,5-Pad3)
- LD9,5 pad 5: Net-(LD10,5-Pad2) -> Net-(LD8,5-Pad2)
Routing:
- net GNDPWR: track 745.8 -> 3524.0 mm, vias 2 -> 10
- net Net-(LD0,5-Pad5): track 0.00 -> 449.5 mm
- net Net-(LD0,5-Pad4): track 4.41 -> 448.0 mm, vias 1 -> 0
- net Net-(LD0,2-Pad5): track 7.11 -> 437.2 mm, vias 1 -> 0
- net Net-(LD0,2-Pad4): track 5.68 -> 435.0 mm, vias 1 -> 0
- net Net-(LD0,4-Pad5): track 0.00 -> 413.5 mm
- net Net-(LD0,4-Pad4): track 0.00 -> 411.1 mm
- net Net-(LD0,3-Pad4): track 0.02 -> 277.1 mm
- net Net-(LD0,3-Pad5): track 5.85 -> 278.9 mm, vias 1 -> 0
- net Net-(LD14,6-Pad5): track 0.00 -> 119.3 mm
- net Net-(LD14,6-Pad4): track 0.00 -> 117.5 mm
- net Net-(LD11,5-Pad3): track 0.00 -> 50.8 mm
- net Net-(LD11,5-Pad2): track 0.00 -> 50.8 mm
- net Net-(LD15,5-Pad2): track 0.00 -> 42.0 mm
- net Net-(LD15,5-Pad3): track 0.00 -> 42.0 mm
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Other:
- board size 448.3 x 179.1 mm -> 444.5 x 179.1 mm
