File: KiCAD/key_matrix.sch (KiCad schematic (older format))
At the start: 232 parts, among them K0,0 KEYSW, K0,1 KEYSW, K0,2 KEYSW, K0,3 KEYSW, K0,4 KEYSW, K0,5 KEYSW, K1,0 KEYSW, K1,1 KEYSW, K1,2 KEYSW, K1,3 KEYSW, K1,4 KEYSW, K1,5 KEYSW, K10,0 KEYSW, K10,1 KEYSW, K10,2 KEYSW, K10,3 KEYSW, K10,4 KEYSW, K10,5 KEYSW, K11,0 KEYSW, K11,1 KEYSW, K11,2 KEYSW, K11,3 KEYSW, K11,4 KEYSW, K11,5 KEYSW, K12,0 KEYSW, K12,1 KEYSW, K12,2 KEYSW, K12,3 KEYSW, K13,1 KEYSW, K13,2 KEYSW, K14,0 KEYSW, K14,1 KEYSW, K14,2 KEYSW, K14,3 KEYSW, K14,4 KEYSW, K14,5 KEYSW, K14,6 KEYSW, K15,0 KEYSW, K15,1 KEYSW, K15,2 KEYSW, K15,3 KEYSW, K15,4 KEYSW, K15,5 KEYSW, K15,6 KEYSW, K16,0 KEYSW, K16,1 KEYSW, K16,2 KEYSW, K16,3 KEYSW, K16,4 KEYSW, K16,5 KEYSW, K16,6 KEYSW, K17,0 KEYSW, K17,1 KEYSW, K17,2 KEYSW, K17,3 KEYSW, K17,4 KEYSW, K17,5 KEYSW, K17,6 KEYSW, K18,0 KEYSW, K18,1 KEYSW, K18,2 KEYSW, K18,3 KEYSW, K18,4 KEYSW, K18,5 KEYSW, K18,6 KEYSW, K19,0 KEYSW, K19,1 KEYSW, K19,2 KEYSW, K19,3 KEYSW, K19,4 KEYSW, K19,5 KEYSW, K19,6 KEYSW, K2,0 KEYSW, K2,1 KEYSW, K2,2 KEYSW, K2,3 KEYSW, K2,4 KEYSW, K2,5 KEYSW, K3,0 KEYSW, K3,1 KEYSW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

Commit message: Update KiCAD files
Parts:
- removed D0,63, D0,65, D0,66, D0,69, D0,71, D0,75, D0,81, D0,87, D0,93, D0,96: D, keyboard_parts:D_SOD123_axial, symbol keyboard_parts:D
- removed K14,2, K14,4, K14,5, K15,2, K15,4, K16,2, K17,2, K18,2, K19,2, K19,5: KEYSW, Switch_Keyboard_Kailh:SW_Hotswap_Kailh_1.00u, symbol keyboard_parts:KEYSW
- added D20,0, D20,1: D, keyboard_parts:D_SOD123_axial, symbol keyboard_parts:D
- added K20,0, K20,1: KEYSW, Switch_Keyboard_Kailh:SW_Hotswap_Kailh_1.00u, symbol keyboard_parts:KEYSW
- renumbered D0,2 to D0,1, D0,3 to D0,2, D0,1 to D0,3, D0,7 to D0,5, D0,11 to D1,4, D0,12 to D1,5, D1,4 to D10,0, D1,5 to D10,1, D1,6 to D10,2, D0,5 to D10,4, D0,6 to D10,5, D2,1 to D11,0, D0,10 to D11,1, D0,51 to D11,2, D0,52 to D11,3, D0,53 to D11,4, D0,54 to D11,5, D3,1 to D12,0, D0,55 to D12,1, D0,56 to D12,2, D0,57 to D12,3, D0,60 to D13,1, D0,61 to D13,2, D5,1 to D14,0, D0,62 to D14,1, D0,64 to D14,3, D0,67 to D14,66, D6,1 to D15,0, D0,68 to D15,1, D0,70 to D15,3, D0,72 to D15,5, D0,73 to D15,6, D7,1 to D16,0, D0,74 to D16,1, D0,76 to D16,3, D0,77 to D16,4, D0,78 to D16,5, D0,79 to D16,6, D5,2 to D17,0, D0,80 to D17,1, D0,82 to D17,3, D0,83 to D17,4, D0,84 to D17,5, D0,85 to D17,6, D6,2 to D18,0, D0,86 to D18,1, D0,88 to D18,3, D0,89 to D18,4, D0,90 to D18,5, D0,91 to D18,6, D7,2 to D19,0, D0,92 to D19,1, D0,94 to D19,3, D0,95 to D19,4, D0,97 to D19,6, D0,8 to D2,1, D0,9 to D2,2, D0,13 to D2,3, D0,14 to D2,4, D0,15 to D2,5, D0,16 to D3,1, D0,17 to D3,2, D0,18 to D3,3, D0,19 to D3,4, D0,20 to D3,5, D0,21 to D4,1, D0,22 to D4,2, D0,23 to D4,3, D0,24 to D4,4, D0,26 to D5,1, D0,27 to D5,2, D0,28 to D5,3, D0,29 to D5,4, D0,31 to D6,1, D0,32 to D6,2, D0,33 to D6,3, D0,34 to D6,4, D0,36 to D7,1, D0,37 to D7,2, D0,38 to D7,3, D0,39 to D7,4, D0,41 to D8,1, D0,42 to D8,2, D0,43 to D8,3, D0,44 to D8,4, D0,45 to D8,5, D0,46 to D9,1, D0,47 to D9,2, D0,48 to D9,3, D0,49 to D9,4, D0,50 to D9,5
Connections:
- net KEY_ROW6: no longer D14,66.1, D15,6.1, D16,6.1, D17,6.1, D18,6.1, D19,6.1
- net at D0,0.1, D1,0.1, D10,0.1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: now also D14,0.1, D15,0.1, D16,0.1, D17,0.1, D18,0.1, D19,0.1, D20,0.1
- net at D0,1.1, D1,1.1, D10,1.1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: now also D14,1.1, D15,1.1, D16,1.1, D17,1.1, D18,1.1, D19,1.1, D20,1.1
- net at D0,3.1, D1,3.1, D10,3.1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: now also D14,3.1, D15,3.1, D16,3.1, D17,3.1, D18,3.1, D19,3.1
- net at D0,4.1, D1,4.1, D10,4.1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: now also D16,4.1, D17,4.1, D18,4.1, D19,4.1
- net at D0,5.1, D1,5.1, D2,5.1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: now also D10,5.1, D11,5.1, D15,5.1, D16,5.1, D17,5.1, D18,5.1, D8,5.1, D9,5.1
- new net: D14,66.1, D15,6.1, D16,6.1, D17,6.1, D18,6.1, D19,6.1
- new net: K20,0.1, K20,1.1
- new net: D20,1.2, K20,1.2
- new net: D20,0.2, K20,0.2
Other:
- moved on the sheet: D0,0, D0,1, D0,2, D0,3, D0,4, D0,5, D1,0, D1,1, D1,2, D1,3, D1,4, D1,5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

Commit message: Update KiCAD files
Parts:
- K0,2: footprint Switch_Keyboard_Kailh:SW_Hotswap_Kailh_1.00u -> Switch_Keyboard_Kailh:SW_Hotswap_Kailh_1.50u
- K0,3: footprint Switch_Keyboard_Kailh:SW_Hotswap_Kailh_1.00u -> Switch_Keyboard_Kailh:SW_Hotswap_Kailh_1.75u
- K0,4: footprint Switch_Keyboard_Kailh:SW_Hotswap_Kailh_1.00u -> Switch_Keyboard_Kailh:SW_Hotswap_Kailh_2.25u
- K17,6: footprint Switch_Keyboard_Kailh:SW_Hotswap_Kailh_1.00u -> Switch_Keyboard_Kailh:SW_Hotswap_Kailh_2.00u
- K19,4, K19,6: footprint Switch_Keyboard_Kailh:SW_Hotswap_Kailh_1.00u -> Switch_Keyboard_Kailh:SW_Hotswap_Kailh_2.00u_Rotated
Changed lines of the file:
@@
 F 0 "K0,2" H 1750 5983 60  0000 C CNN
 F 1 "KEYSW" H 1750 5650 60  0001 C CNN
-F 2 "Switch_Keyboard_Kailh:SW_Hotswap_Kailh_1.00u" H 1750 5983 60  0001 C CNN
+F 2 "Switch_Keyboard_Kailh:SW_Hotswap_Kailh_1.50u" H 1750 5983 60  0001 C CNN
 F 3 "" H 1750 5750 60  0000 C CNN
 	1    1750 5750
@@
 F 0 "K0,3" H 1750 6733 60  0000 C CNN
 F 1 "KEYSW" H 1750 6400 60  0001 C CNN
-F 2 "Switch_Keyboard_Kailh:SW_Hotswap_Kailh_1.00u" H 1750 6733 60  0001 C CNN
+F 2 "Switch_Keyboard_Kailh:SW_Hotswap_Kailh_1.75u" H 1750 6733 60  0001 C CNN
 F 3 "" H 1750 6500 60  0000 C CNN
 	1    1750 6500
@@
 F 0 "K0,4" H 1750 7483 60  0000 C CNN
 F 1 "KEYSW" H 1750 7150 60  0001 C CNN
-F 2 "Switch_Keyboard_Kailh:SW_Hotswap_Kailh_1.00u" H 1750 7483 60  0001 C CNN
+F 2 "Switch_Keyboard_Kailh:SW_Hotswap_Kailh_2.25u" H 1750 7483 60  0001 C CNN
 F 3 "" H 1750 7250 60  0000 C CNN
 	1    1750 7250
@@
 F 0 "K19,6" H 19000 8983 60  0000 C CNN
 F 1 "KEYSW" H 19000 8650 60  0001 C CNN
-F 2 "Switch_Keyboard_Kailh:SW_Hotswap_Kailh_1.00u" H 19000 8983 60  0001 C CNN
+F 2 "Switch_Keyboard_Kailh:SW_Hotswap_Kailh_2.00u_Rotated" H 19000 8983 60  0001 C CNN
 F 3 "" H 19000 8750 60  0000 C CNN
 	1    19000 8750
@@
 F 0 "K17,6" H 17300 8983 60  0000 C CNN
 F 1 "KEYSW" H 17300 8650 60  0001 C CNN
-F 2 "Switch_Keyboard_Kailh:SW_Hotswap_Kailh_1.00u" H 17300 8983 60  0001 C CNN
+F 2 "Switch_Keyboard_Kailh:SW_Hotswap_Kailh_2.00u" H 17300 8983 60  0001 C CNN
 F 3 "" H 17300 8750 60  0000 C CNN
 	1    17300 8750
@@
 F 0 "K19,4" H 19000 7483 60  0000 C CNN
 F 1 "KEYSW" H 19000 7150 60  0001 C CNN
-F 2 "Switch_Keyboard_Kailh:SW_Hotswap_Kailh_1.00u" H 19000 7483 60  0001 C CNN
+F 2 "Switch_Keyboard_Kailh:SW_Hotswap_Kailh_2.00u_Rotated" H 19000 7483 60  0001 C CNN
 F 3 "" H 19000 7250 60  0000 C CNN
 	1    19000 7250

Commit message: Update KiCAD files
Parts:
- renumbered D14,66 to D14,6
Connections:
- net KEY_COL0: now also K0,0.1, K0,1.1, K0,2.1, K0,3.1, K0,4.1, K0,5.1
- net KEY_COL1: now also K1,0.1, K1,1.1, K1,2.1, K1,3.1, K1,4.1, K1,5.1
- net KEY_COL10: now also K10,0.1, K10,1.1, K10,2.1, K10,3.1, K10,4.1, K10,5.1
- net KEY_COL11: now also K11,0.1, K11,1.1, K11,2.1, K11,3.1, K11,4.1, K11,5.1
- net KEY_COL12: now also K12,0.1, K12,1.1, K12,2.1, K12,3.1
- net KEY_COL13: now also K13,1.1, K13,2.1
- net KEY_COL14: now also K14,0.1, K14,1.1, K14,3.1, K14,6.1
- net KEY_COL15: now also K15,0.1, K15,1.1, K15,3.1, K15,5.1, K15,6.1
- net KEY_COL16: now also K16,0.1, K16,1.1, K16,3.1, K16,4.1, K16,5.1, K16,6.1
- net KEY_COL17: now also K17,0.1, K17,1.1, K17,3.1, K17,4.1, K17,5.1, K17,6.1
- net KEY_COL18: now also K18,0.1, K18,1.1, K18,3.1, K18,4.1, K18,5.1, K18,6.1
- net KEY_COL19: now also K19,0.1, K19,1.1, K19,3.1, K19,4.1, K19,6.1
- net KEY_COL2: now also K2,0.1, K2,1.1, K2,2.1, K2,3.1, K2,4.1, K2,5.1
- net KEY_COL3: now also K3,0.1, K3,1.1, K3,2.1, K3,3.1, K3,4.1, K3,5.1
- net KEY_COL4: now also K4,0.1, K4,1.1, K4,2.1, K4,3.1, K4,4.1
- net KEY_COL5: now also K5,0.1, K5,1.1, K5,2.1, K5,3.1, K5,4.1
- net KEY_COL6: now also K6,0.1, K6,1.1, K6,2.1, K6,3.1, K6,4.1
- net KEY_COL7: now also K7,0.1, K7,1.1, K7,2.1, K7,3.1, K7,4.1
- net KEY_COL8: now also K8,0.1, K8,1.1, K8,2.1, K8,3.1, K8,4.1, K8,5.1
- net KEY_COL9: now also K9,0.1, K9,1.1, K9,2.1, K9,3.1, K9,4.1, K9,5.1
- net KEY_ROW0: now also D0,0.1, D1,0.1, D10,0.1, D11,0.1, D12,0.1, D14,0.1, D15,0.1, D16,0.1, D17,0.1, D18,0.1, D19,0.1, D2,0.1, D20,0.1, D3,0.1, D4,0.1, D5,0.1, D6,0.1, D7,0.1, D8,0.1, D9,0.1
- net KEY_ROW1: now also D0,1.1, D1,1.1, D10,1.1, D11,1.1, D12,1.1, D13,1.1, D14,1.1, D15,1.1, D16,1.1, D17,1.1, D18,1.1, D19,1.1, D2,1.1, D20,1.1, D3,1.1, D4,1.1, D5,1.1, D6,1.1, D7,1.1, D8,1.1, D9,1.1
- net KEY_ROW2: now also D0,2.1, D1,2.1, D10,2.1, D11,2.1, D12,2.1, D13,2.1, D2,2.1, D3,2.1, D4,2.1, D5,2.1, D6,2.1, D7,2.1, D8,2.1, D9,2.1
- net KEY_ROW3: now also D0,3.1, D1,3.1, D10,3.1, D11,3.1, D12,3.1, D14,3.1, D15,3.1, D16,3.1, D17,3.1, D18,3.1, D19,3.1, D2,3.1, D3,3.1, D4,3.1, D5,3.1, D6,3.1, D7,3.1, D8,3.1, D9,3.1
- net KEY_ROW4: now also D0,4.1, D1,4.1, D10,4.1, D11,4.1, D16,4.1, D17,4.1, D18,4.1, D19,4.1, D2,4.1, D3,4.1, D4,4.1, D5,4.1, D6,4.1, D7,4.1, D8,4.1, D9,4.1
- net KEY_ROW5: now also D0,5.1, D1,5.1, D10,5.1, D11,5.1, D15,5.1, D16,5.1, D17,5.1, D18,5.1, D2,5.1, D3,5.1, D8,5.1, D9,5.1
- net KEY_ROW6: now also D14,6.1, D15,6.1, D16,6.1, D17,6.1, D18,6.1, D19,6.1
- net KEY_COL20: now reaches K20,0.1, K20,1.1
Changed lines of the file:
@@
 	2950 4100 2950 4300
 Connection ~ 2950 4300
-Entry Wire Line
-	2000 4000 2100 4100
-Entry Wire Line
-	2850 4000 2950 4100
-Entry Wire Line
-	3700 4000 3800 4100
-Entry Wire Line
-	1250 5300 1350 5400
-Entry Wire Line
-	1250 6050 1350 6150
-Entry Wire Line
-	1250 4600 1350 4700
 $Comp
 L keyboard_parts:D D3,2
@@
 	1350 6900 1450 6900
 Connection ~ 1450 6900
-Entry Wire Line
-	1250 6800 1350 6900
 $Comp
 L keyboard_parts:D D0,4
@@
 Connection ~ 1450 7650
 Connection ~ 2100 7250
-Entry Wire Line
-	1250 7550 1350 7650
 $Comp
 L keyboard_parts:D D0,5
@@
 	1350 8400 1450 8400
 Connection ~ 1450 8400
-Entry Wire Line
-	1250 8300 1350 8400
 Wire Wire Line
 	4650 4100 4650 4300
-Entry Wire Line
-	4550 4000 4650 4100
 $Comp
 L keyboard_parts:D D4,0
@@
 Wire Wire Line
 	5500 4100 5500 4300
-Entry Wire Line
-	5400 4000 5500 4100
 $Comp
 L keyboard_parts:D D5,0
@@
 Wire Wire Line
 	6350 4100 6350 4300
-Entry Wire Line
-	6250 4000 6350 4100
 $Comp
 L keyboard_parts:D D6,0
@@
 Wire Wire Line
 	7200 4100 7200 4300
-Entry Wire Line
-	7100 4000 7200 4100
 $Comp
 L keyboard_parts:D D7,0
@@
 Wire Wire Line
 	8700 4100 8700 4300
-Entry Wire Line
-	8600 4000 8700 4100
 $Comp
 L keyboard_parts:D D8,0
@@
 Wire Wire Line
 	9550 4100 9550 4300
-Entry Wire Line
-	9450 4000 9550 4100
 $Comp
 L keyboard_parts:D D9,0
@@
 Wire Wire Line
 	10400 4100 10400 4300
-Entry Wire Line
-	10300 4000 10400 4100
 $Comp
 L keyboard_parts:D D5,2
@@
 Wire Wire Line
 	4850 7650 5700 7650
-Text GLabel 2000 4000 0    39   BiDi ~ 0
+Text GLabel 2100 4100 0    39   BiDi ~ 0
 KEY_COL0
-Text GLabel 2850 4000 0    39   BiDi ~ 0
+Text GLabel 2950 4100 0    39   BiDi ~ 0
 KEY_COL1
-Text GLabel 3700 4000 0    39   BiDi ~ 0
+Text GLabel 3800 4100 0    39   BiDi ~ 0
 KEY_COL2
-Text GLabel 4550 4000 0    39   BiDi ~ 0
+Text GLabel 4650 4100 0    39   BiDi ~ 0
 KEY_COL3
-Text GLabel 5400 4000 0    39   BiDi ~ 0
+Text GLabel 5500 4100 0    39   BiDi ~ 0
 KEY_COL4
-Text GLabel 6250 4000 0    39   BiDi ~ 0
+Text GLabel 6350 4100 0    39   BiDi ~ 0
 KEY_COL5
-Text GLabel 7100 4000 0    39   BiDi ~ 0
+Text GLabel 7200 4100 0    39   BiDi ~ 0
 KEY_COL6
-Text GLabel 8600 4000 0    39   BiDi ~ 0
+Text GLabel 8700 4100 0    39   BiDi ~ 0
 KEY_COL7
-Text GLabel 9450 4000 0    39   BiDi ~ 0
+Text GLabel 9550 4100 0    39   BiDi ~ 0
 KEY_COL8
-Text GLabel 10300 4000 0    39   BiDi ~ 0
+Text GLabel 10400 4100 0    39   BiDi ~ 0
 KEY_COL9
-Text GLabel 1250 4600 0    39   BiDi ~ 0
+Text GLabel 1350 4700 0    39   BiDi ~ 0
 KEY_ROW0
-Text GLabel 1250 5300 0    39   BiDi ~ 0
+Text GLabel 1350 5400 0    39   BiDi ~ 0
 KEY_ROW1
-Text GLabel 1250 6050 0    39   BiDi ~ 0
+Text GLabel 1350 6150 0    39   BiDi ~ 0
 KEY_ROW2
-Text GLabel 1250 6800 0    39   BiDi ~ 0
+Text GLabel 1350 6900 0    39   BiDi ~ 0
 KEY_ROW3
-Text GLabel 1250 7550 0    39   BiDi ~ 0
+Text GLabel 1350 7650 0    39   BiDi ~ 0
 KEY_ROW4
-Text GLabel 1250 8300 0    39   BiDi ~ 0
+Text GLabel 1350 8400 0    39   BiDi ~ 0
 KEY_ROW5
 $Comp
@@
 	11250 4100 11250 4300
 Connection ~ 11250 4300
-Entry Wire Line
-	11150 4000 11250 4100
-Entry Wire Line
-	12000 4000 12100 4100
 $Comp
 L keyboard_parts:D D12,2
@@
 Wire Wire Line
 	12950 4100 12950 4300
-Entry Wire Line
-	12850 4000 12950 4100
-Entry Wire Line
-	13700 4000 13800 4100
 $Comp
 L keyboard_parts:D D11,2
@@
 Wire Wire Line
 	12100 7250 12100 8000
-Text GLabel 11150 4000 0    39   BiDi ~ 0
+Text GLabel 11250 4100 0    39   BiDi ~ 0
 KEY_COL10
-Text GLabel 12000 4000 0    39   BiDi ~ 0
+Text GLabel 12100 4100 0    39   BiDi ~ 0
 KEY_COL11
-Text GLabel 12850 4000 0    39   BiDi ~ 0
+Text GLabel 12950 4100 0    39   BiDi ~ 0
 KEY_COL12
-Text GLabel 13700 4000 0    39   BiDi ~ 0
+Text GLabel 13800 4100 0    39   BiDi ~ 0
 KEY_COL13
 Wire Wire Line
@@
 	-1   0    0    1
 $EndComp
-Text GLabel 19250 4000 0    39   BiDi ~ 0
+Text GLabel 19350 4100 0    39   BiDi ~ 0
 KEY_COL19
-Text GLabel 18400 4000 0    39   BiDi ~ 0
+Text GLabel 18500 4100 0    39   BiDi ~ 0
 KEY_COL18
-Text GLabel 17550 4000 0    39   BiDi ~ 0
+Text GLabel 17650 4100 0    39   BiDi ~ 0
 KEY_COL17
 Wire Wire Line
@@
 	-1   0    0    1
 $EndComp
-Entry Wire Line
-	19250 4000 19350 4100
 Wire Wire Line
 	19350 4100 19350 4300
@@
 	-1   0    0    1
 $EndComp
-Entry Wire Line
-	18400 4000 18500 4100
 Wire Wire Line
 	18500 4100 18500 4300
@@
 	-1   0    0    1
 $EndComp
-Entry Wire Line
-	17550 4000 17650 4100
 Wire Wire Line
 	17650 4100 17650 4300
@@
 $EndComp
 $Comp
-L keyboard_parts:D D14,66
+L keyboard_parts:D D14,6
 U 1 1 61C5EF26
 P 14450 9000
-F 0 "D14,66" H 14322 8950 60  0000 R CNN
+F 0 "D14,6" H 14322 8950 60  0000 R CNN
 F 1 "D" V 14600 8950 60  0001 C CNN
 F 2 "keyboard_parts:D_SOD123_axial" H 14322 9003 60  0001 R CNN
@@
 	-1   0    0    1
 $EndComp
-Text GLabel 14250 9100 0    20   BiDi ~ 0
+Text GLabel 14250 9150 0    20   BiDi ~ 0
 KEY_ROW6
-Text GLabel 16700 4000 0    39   BiDi ~ 0
+Text GLabel 16800 4100 0    39   BiDi ~ 0
 KEY_COL16
-Text GLabel 15850 4000 0    39   BiDi ~ 0
+Text GLabel 15950 4100 0    39   BiDi ~ 0
 KEY_COL15
-Text GLabel 15000 4000 0    39   BiDi ~ 0
+Text GLabel 15100 4100 0    39   BiDi ~ 0
 KEY_COL14
 Wire Wire Line
@@
 	-1   0    0    1
 $EndComp
-Entry Wire Line
-	16700 4000 16800 4100
 Wire Wire Line
 	16800 4100 16800 4300
@@
 	-1   0    0    1
 $EndComp
-Entry Wire Line
-	15850 4000 15950 4100
 Wire Wire Line
 	15950 4100 15950 4300
@@
 	-1   0    0    1
 $EndComp
-Entry Wire Line
-	15000 4000 15100 4100
 Wire Wire Line
 	15100 4100 15100 4300
@@
 Connection ~ 19350 5000
 Connection ~ 19350 6500
-Text GLabel 20100 4000 0    39   BiDi ~ 0
-KEY_COL19
+Text GLabel 20200 4100 0    39   BiDi ~ 0
+KEY_COL20
 Wire Wire Line
 	18700 5400 19550 5400
@@
 	-1   0    0    1
 $EndComp
-Entry Wire Line
-	20100 4000 20200 4100
 Wire Wire Line
 	20200 4100 20200 4300

Commit message: Update KiCAD files
Parts:
- D12,2: value D -> BAT54W-HG3-18

Commit message: Update KiCAD files.
Parts:
- D0,0, D0,1, D0,2, D0,3, D0,4, D0,5, D1,0, D1,1, D1,2, D1,3, D1,4, D1,5, D10,0, D10,1, D10,2, D10,3, D10,4, D10,5, D11,0, D11,1, D11,2, D11,3, D11,4, D11,5, D12,0, D12,1, D12,3, D13,1, D13,2, D14,0, D14,1, D14,3, D14,6, D15,0, D15,1, D15,3, D15,5, D15,6, D16,0, D16,1, D16,3, D16,4, D16,5, D16,6, D17,0, D17,1, D17,3, D17,4, D17,5, D17,6, D18,0, D18,1, D18,3, D18,4, D18,5, D18,6, D19,0, D19,1, D19,3, D19,4, D19,6, D2,0, D2,1, D2,2, D2,3, D2,4, D2,5, D20,0, D20,1, D3,0, D3,1, D3,2, D3,3, D3,4, D3,5, D4,0, D4,1, D4,2, D4,3, D4,4, D5,0, D5,1, D5,2, D5,3, D5,4, D6,0, D6,1, D6,2, D6,3, D6,4, D7,0, D7,1, D7,2, D7,3, D7,4, D8,0, D8,1, D8,2, D8,3, D8,4, D8,5, D9,0, D9,1, D9,2, D9,3, D9,4, D9,5: value D -> BAT54W-HG3-08; Mouser No (none) -> 78-BAT54W-HG3-08
- D12,2: value BAT54W-HG3-18 -> BAT54W-HG3-08; Mouser No (none) -> 78-BAT54W-HG3-08
- K0,0, K0,1, K0,2, K0,3, K0,4, K0,5, K1,0, K1,1, K1,2, K1,3, K1,4, K1,5, K10,0, K10,1, K10,2, K10,3, K10,4, K10,5, K11,0, K11,1, K11,2, K11,3, K11,4, K11,5, K12,0, K12,1, K12,2, K12,3, K13,1, K13,2, K14,0, K14,1, K14,3, K14,6, K15,0, K15,1, K15,3, K15,5, K15,6, K16,0, K16,1, K16,3, K16,4, K16,5, K16,6, K17,0, K17,1, K17,3, K17,4, K17,5, K17,6, K18,0, K18,1, K18,3, K18,4, K18,5, K18,6, K19,0, K19,1, K19,3, K19,4, K19,6, K2,0, K2,1, K2,2, K2,3, K2,4, K2,5, K20,0, K20,1, K3,0, K3,1, K3,2, K3,3, K3,4, K3,5, K4,0, K4,1, K4,2, K4,3, K4,4, K5,0, K5,1, K5,2, K5,3, K5,4, K6,0, K6,1, K6,2, K6,3, K6,4, K7,0, K7,1, K7,2, K7,3, K7,4, K8,0, K8,1, K8,2, K8,3, K8,4, K8,5, K9,0, K9,1, K9,2, K9,3, K9,4, K9,5: value KEYSW -> ~

Commit message: Update KiCAD and firmware files. Firmware has had a little bit of work to make sending key data easier. PCB has been fully routed for the 4th time and should be good to test LEDs and a much more populated board.
Parts:
- D0,0, D0,1, D0,2, D0,3, D0,4, D0,5, D1,0, D1,1, D1,2, D1,3, D1,4, D1,5, D10,0, D10,1, D10,2, D10,3, D10,4, D10,5, D11,0, D11,1, D11,2, D11,3, D11,4, D11,5, D12,0, D12,1, D12,2, D12,3, D13,1, D13,2, D14,0, D14,1, D14,3, D14,6, D15,0, D15,1, D15,3, D15,5, D15,6, D16,0, D16,1, D16,3, D16,4, D16,5, D16,6, D17,0, D17,1, D17,3, D17,4, D17,5, D17,6, D18,0, D18,1, D18,3, D18,4, D18,5, D18,6, D19,0, D19,1, D19,3, D19,4, D19,6, D2,0, D2,1, D2,2, D2,3, D2,4, D2,5, D20,0, D20,1, D3,0, D3,1, D3,2, D3,3, D3,4, D3,5, D4,0, D4,1, D4,2, D4,3, D4,4, D5,0, D5,1, D5,2, D5,3, D5,4, D6,0, D6,1, D6,2, D6,3, D6,4, D7,0, D7,1, D7,2, D7,3, D7,4, D8,0, D8,1, D8,2, D8,3, D8,4, D8,5, D9,0, D9,1, D9,2, D9,3, D9,4, D9,5: value BAT54W-HG3-08 -> 1N4148W-7-F; Mouser No 78-BAT54W-HG3-08 -> 621-1N4148W-F
