File: KiCAD/led_strings.sch (KiCad schematic (older format))
At the start: 115 parts

Commit message: Update KiCAD and firmware files. Firmware has had a little bit of work to make sending key data easier. PCB has been fully routed for the 4th time and should be good to test LEDs and a much more populated board.
Connections:
- net at LD3,5,0.2 (CKO): now also LD3,5.5 (CKI); no longer LD2,5.5 (CKI)
- net at LD3,5,0.3 (SDO): now also LD3,5.4 (SDI); no longer LD2,5.4 (SDI)
- net at LD3,5,0.4 (SDI): now also LD2,5.3 (SDO); no longer LD3,5.3 (SDO)
- net at LD3,5,0.5 (CKI): now also LD2,5.2 (CKO); no longer LD3,5.2 (CKO)
- net at LD3,5,1.2 (CKO): now also LD8,5.5 (CKI); no longer LD3,5.5 (CKI)
- net at LD3,5,1.3 (SDO): now also LD8,5.4 (SDI); no longer LD3,5.4 (SDI)
- net at LD3,5,1.4 (SDI): now also LD3,5.3 (SDO); no longer LD8,5.3 (SDO)
- net at LD3,5,1.5 (CKI): now also LD3,5.2 (CKO); no longer LD8,5.2 (CKO)
- net at LD14,6.4 (SDI): now also LD18,5.3 (SDO); no longer LD0,5.3 (SDO)
- net at LD14,6.5 (CKI): now also LD18,5.2 (CKO); no longer LD0,5.2 (CKO)
- net at LD13,2.2 (CKO): now also LD0,3.5 (CKI); no longer LD19,3.5 (CKI)
- net at LD13,2.3 (SDO): now also LD0,3.4 (SDI); no longer LD19,3.4 (SDI)
- net at LD0,3.2 (CKO): now also LD1,3.5 (CKI); no longer LD0,4.5 (CKI)
- net at LD0,3.3 (SDO): now also LD1,3.4 (SDI); no longer LD0,4.4 (SDI)
- net at LD1,3.3 (SDO): now also LD2,3.4 (SDI); no longer LD0,3.4 (SDI)
- net at LD1,3.2 (CKO): now also LD2,3.5 (CKI); no longer LD0,3.5 (CKI)
- net at LD2,3.3 (SDO): now also LD3,3.4 (SDI); no longer LD1,3.4 (SDI)
- net at LD2,3.2 (CKO): now also LD3,3.5 (CKI); no longer LD1,3.5 (CKI)
- net at LD3,3.3 (SDO): now also LD4,3.4 (SDI); no longer LD2,3.4 (SDI)
- net at LD3,3.2 (CKO): now also LD4,3.5 (CKI); no longer LD2,3.5 (CKI)
- net at LD4,3.3 (SDO): now also LD5,3.4 (SDI); no longer LD3,3.4 (SDI)
- net at LD4,3.2 (CKO): now also LD5,3.5 (CKI); no longer LD3,3.5 (CKI)
- net at LD5,3.3 (SDO): now also LD6,3.4 (SDI); no longer LD4,3.4 (SDI)
- net at LD5,3.2 (CKO): now also LD6,3.5 (CKI); no longer LD4,3.5 (CKI)
- net at LD6,3.3 (SDO): now also LD7,3.4 (SDI); no longer LD5,3.4 (SDI)
- net at LD6,3.2 (CKO): now also LD7,3.5 (CKI); no longer LD5,3.5 (CKI)
- net at LD7,3.3 (SDO): now also LD8,3.4 (SDI); no longer LD6,3.4 (SDI)
- net at LD7,3.2 (CKO): now also LD8,3.5 (CKI); no longer LD6,3.5 (CKI)
- net at LD8,3.3 (SDO): now also LD9,3.4 (SDI); no longer LD7,3.4 (SDI)
- net at LD8,3.2 (CKO): now also LD9,3.5 (CKI); no longer LD7,3.5 (CKI)
- net at LD9,3.3 (SDO): now also LD10,3.4 (SDI); no longer LD8,3.4 (SDI)
- net at LD9,3.2 (CKO): now also LD10,3.5 (CKI); no longer LD8,3.5 (CKI)
- net at LD10,3.3 (SDO): now also LD11,3.4 (SDI); no longer LD9,3.4 (SDI)
- net at LD10,3.2 (CKO): now also LD11,3.5 (CKI); no longer LD9,3.5 (CKI)
- net at LD11,3.3 (SDO): now also LD12,3.4 (SDI); no longer LD10,3.4 (SDI)
- net at LD11,3.2 (CKO): now also LD12,3.5 (CKI); no longer LD10,3.5 (CKI)
- net at LD12,3.3 (SDO): now also LD14,3.4 (SDI); no longer LD11,3.4 (SDI)
- net at LD12,3.2 (CKO): now also LD14,3.5 (CKI); no longer LD11,3.5 (CKI)
- net at LD14,3.3 (SDO): now also LD15,3.4 (SDI); no longer LD12,3.4 (SDI)
- net at LD14,3.2 (CKO): now also LD15,3.5 (CKI); no longer LD12,3.5 (CKI)
- net at LD15,3.3 (SDO): now also LD16,3.4 (SDI); no longer LD14,3.4 (SDI)
- net at LD15,3.2 (CKO): now also LD16,3.5 (CKI); no longer LD14,3.5 (CKI)
- net at LD16,3.3 (SDO): now also LD17,3.4 (SDI); no longer LD15,3.4 (SDI)
- net at LD16,3.2 (CKO): now also LD17,3.5 (CKI); no longer LD15,3.5 (CKI)
- net at LD17,3.3 (SDO): now also LD18,3.4 (SDI); no longer LD16,3.4 (SDI)
- net at LD17,3.2 (CKO): now also LD18,3.5 (CKI); no longer LD16,3.5 (CKI)
- net at LD18,3.3 (SDO): now also LD19,3.4 (SDI); no longer LD17,3.4 (SDI)
- net at LD18,3.2 (CKO): now also LD19,3.5 (CKI); no longer LD17,3.5 (CKI)
- net at LD19,3.3 (SDO): now also LD0,4.4 (SDI); no longer LD18,3.4 (SDI)
- net at LD19,3.2 (CKO): now also LD0,4.5 (CKI); no longer LD18,3.5 (CKI)
- net at LD19,4.2 (CKO): now also LD0,5.5 (CKI); no longer LD18,5.5 (CKI)
- net at LD19,4.3 (SDO): now also LD0,5.4 (SDI); no longer LD18,5.4 (SDI)
- net at LD1,5.3 (SDO): now also LD2,5.4 (SDI); no longer LD0,5.4 (SDI)
- net at LD1,5.2 (CKO): now also LD2,5.5 (CKI); no longer LD0,5.5 (CKI)
- net at LD1,5.4 (SDI): now also LD0,5.3 (SDO); no longer LD2,5.3 (SDO)
- net at LD1,5.5 (CKI): now also LD0,5.2 (CKO); no longer LD2,5.2 (CKO)
- net at LD9,5.3 (SDO): now also LD10,5.4 (SDI); no longer LD8,5.4 (SDI)
- net at LD9,5.2 (CKO): now also LD10,5.5 (CKI); no longer LD8,5.5 (CKI)
- net at LD9,5.4 (SDI): now also LD8,5.3 (SDO); no longer LD10,5.3 (SDO)
- net at LD9,5.5 (CKI): now also LD8,5.2 (CKO); no longer LD10,5.2 (CKO)
- net at LD11,5.3 (SDO): now also LD15,5.4 (SDI); no longer LD10,5.4 (SDI)
- net at LD11,5.2 (CKO): now also LD15,5.5 (CKI); no longer LD10,5.5 (CKI)
- net at LD11,5.4 (SDI): now also LD10,5.3 (SDO); no longer LD15,5.3 (SDO)
- net at LD11,5.5 (CKI): now also LD10,5.2 (CKO); no longer LD15,5.2 (CKO)
- net at LD16,5.3 (SDO): now also LD17,5.4 (SDI); no longer LD15,5.4 (SDI)
- net at LD16,5.2 (CKO): now also LD17,5.5 (CKI); no longer LD15,5.5 (CKI)
- net at LD16,5.4 (SDI): now also LD15,5.3 (SDO); no longer LD17,5.3 (SDO)
- net at LD16,5.5 (CKI): now also LD15,5.2 (CKO); no longer LD17,5.2 (CKO)
- new net: LD17,5.2 (CKO), LD18,5.5 (CKI)
- new net: LD17,5.3 (SDO), LD18,5.4 (SDI)
Other:
- moved on the sheet: LD0,3, LD0,5, LD1,3, LD1,5, LD10,3, LD10,5, LD11,3, LD11,5, LD12,3, LD14,3, LD15,3, LD15,5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
