File: KiCAD/Mainboard/RedPyKeeb_mainboard.kicad_pcb (KiCad board)
At the start: 4 copper layers, 440.7 x 154.9 mm, 332 parts, among them J1 Conn_01x36

Commit message: Firmware is as-is for now, I've been testing PCB revisions and seeing what kind of latency I can poll the entire key matrix at KiCAD designs are looking really good now and I shoulld have parts in the next few weeks that will let me validate the keyboard as a whole plus the firmware.
Routing:
- net LED_SCL_ROW0: track 2.64 -> 355.0 mm
- net LED_SDA_ROW0: track 0.00 -> 349.0 mm
- net LED_SDA_STATUS0: track 3.49 -> 139.1 mm
- net LED_SCL_STATUS0: track 53.0 -> 138.7 mm
- net KEY_ROW0: track 564.8 -> 548.8 mm
- net KEY_ROW1: track 562.9 -> 554.4 mm
- net KEY_COL20: track 93.4 -> 88.4 mm
- added copper zone on MISC, net GNDPWR
- added copper zone on PWRGND, net GNDPWR

Commit message: Latest KiCAD files and what ever I had for testing the old boards.
Parts:
- removed K18,0: ~, Switch_Keyboard_Kailh:SW_Hotswap_Kailh_1.00u
- J1: value Conn_01x36 -> Conn_02x20_Top_Bottom; footprint Connector_PinHeader_2.00mm:PinHeader_1x36_P2.00mm_Horizontal -> Connector_PinHeader_2.54mm:PinHeader_2x20_P2.54mm_Vertical_SMD
- moved J1 27.3 mm to (368.4, 24.3)
Connections:
- J1 pad 10: LED_SCL_ROW0 -> KEY_COL2
- J1 pad 11: GNDPWR -> KEY_COL3
- J1 pad 12: KEY_COL0 -> KEY_COL4
- J1 pad 13: KEY_COL1 -> KEY_COL5
- J1 pad 14: KEY_COL2 -> KEY_COL6
- J1 pad 15: KEY_COL3 -> KEY_COL7
- J1 pad 16: KEY_COL4 -> KEY_COL8
- J1 pad 17: KEY_COL5 -> KEY_COL9
- J1 pad 18: KEY_COL6 -> KEY_COL10
- J1 pad 19: KEY_COL7 -> KEY_COL11
- J1 pad 20: KEY_COL8 -> KEY_COL12
- J1 pad 21: KEY_COL9 -> LED_SDA_ROW0
- J1 pad 22: KEY_COL10 -> LED_SCL_ROW0
- J1 pad 23: KEY_COL11 -> KEY_COL13
- J1 pad 24: KEY_COL12 -> KEY_COL14
- J1 pad 25: KEY_COL13 -> KEY_COL15
- J1 pad 26: KEY_COL14 -> KEY_COL16
- J1 pad 27: KEY_COL15 -> KEY_COL17
- J1 pad 28: KEY_COL16 -> KEY_COL18
- J1 pad 29: KEY_COL17 -> KEY_COL19
- J1 pad 30: KEY_COL18 -> KEY_COL20
- J1 pad 31: KEY_COL19 -> Net-(J1-Pad31)
- J1 pad 32: KEY_COL20 -> Net-(J1-Pad32)
- J1 pad 33: MAIN_VBUS -> Net-(J1-Pad33)
- J1 pad 34: LED_SDA_STATUS0 -> Net-(J1-Pad34)
- J1 pad 35: LED_SCL_STATUS0 -> GNDPWR
- J1 pad 8: MAIN_VBUS -> KEY_COL0
- J1 pad 9: LED_SDA_ROW0 -> KEY_COL1
- LD19,6 pad 2: (no net) -> Net-(LD19,6-Pad2)
- LD19,6 pad 3: (no net) -> Net-(LD19,6-Pad3)
- LD20,7 pad 2: (no net) -> Net-(LD20,7-Pad2)
- LD20,7 pad 3: (no net) -> Net-(LD20,7-Pad3)
Routing:
- net MAIN_VBUS: track 4299.7 -> 53.4 mm, vias 50 -> 4
- net GNDPWR: track 3495.5 -> 68.3 mm
- net KEY_COL15: track 226.4 -> 162.3 mm, vias 1 -> 2
- net KEY_COL20: track 88.4 -> 115.9 mm, vias 1 -> 2
- net KEY_COL18: track 142.5 -> 168.8 mm, vias 1 -> 2
- net LED_SDA_ROW0: track 349.0 -> 374.5 mm
- net KEY_COL19: track 153.4 -> 175.6 mm, vias 1 -> 2
- net LED_SCL_STATUS0: track 138.7 -> 159.9 mm
- net LED_SCL_ROW0: track 355.0 -> 374.0 mm
- net LED_SDA_STATUS0: track 139.1 -> 156.0 mm
- net KEY_COL13: track 167.9 -> 153.1 mm, vias 0 -> 1
- net Net-(LD0,5-Pad4): track 448.0 -> 460.8 mm
- net Net-(LD0,5-Pad5): track 449.5 -> 462.1 mm
- net KEY_COL7: track 321.6 -> 309.5 mm, vias 0 -> 1
- net KEY_ROW3: track 465.2 -> 476.7 mm
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- added copper zone on GND, net GNDPWR
- added copper zone on PWR, net MAIN_VBUS
- removed copper zone on MISC, net GNDPWR
- removed copper zone on PWRGND, net GNDPWR

Commit message: NKRO is now supported and I've got what I believe to be working PCBs now
Routing:
- net LED_SDA_ROW0: track 374.5 -> 376.1 mm
- net LED_SCL_ROW0: track 374.0 -> 374.7 mm
- net KEY_ROW0: track 554.3 -> 554.9 mm

Commit message: Minimum viable product! I still need to work out a few things on the PCBs but its finally real!
Parts:
- added C6: EEE-FN1C102UV, Capacitor_SMD:CP_Elec_10x10, F.Cu at (430.3, 25.4)
- added K18,0: ~, Switch_Keyboard_Kailh:SW_Hotswap_Kailh_1.00u, F.Cu at (400.5, 55.5)
Routing:
- net KEY_ROW6: track 320.3 -> 317.4 mm
- net KEY_ROW5: track 581.8 -> 580.5 mm

Commit message: Add dip switch to allow for plug-in/boot time option selects. Add status light LEDs to be handled and actually reflect capslock and numlock status. Add tiny debounce which is enough on my prototype board to remove false-positive key registration on the first column.
Parts:
- D0,0, D0,1, D0,2, D0,3, D0,4, D0,5, D1,0, D1,1, D1,2, D1,3, D1,4, D1,5, D10,0, D10,1, D10,2, D10,3, D10,4, D10,5, D11,0, D11,1, D11,2, D11,3, D11,4, D11,5, D12,0, D12,1, D12,2, D12,3, D13,1, D13,2, D14,0, D14,1, D14,3, D14,6, D15,0, D15,1, D15,3, D15,5, D15,6, D16,0, D16,1, D16,3, D16,4, D16,5, D16,6, D17,0, D17,1, D17,3, D17,4, D17,5, D17,6, D18,0, D18,1, D18,3, D18,4, D18,5, D18,6, D19,0, D19,1, D19,3, D19,4, D19,6, D2,0, D2,1, D2,2, D2,3, D2,4, D2,5, D20,0, D20,1, D3,0, D3,1, D3,2, D3,3, D3,4, D3,5, D4,0, D4,1, D4,2, D4,3, D4,4, D5,0, D5,1, D5,2, D5,3, D5,4, D6,0, D6,1, D6,2, D6,3, D6,4, D7,0, D7,1, D7,2, D7,3, D7,4, D8,0, D8,1, D8,2, D8,3, D8,4, D8,5, D9,0, D9,1, D9,2, D9,3, D9,4, D9,5: moved to F.Cu
- J1: footprint Connector_PinHeader_2.54mm:PinHeader_2x20_P2.54mm_Vertical_SMD -> Custom_pico:PinHeader_2x20_P2.54mm_Vertical_SMD_doublesided
Routing:
- net Net-(LD0,4-Pad5): track 413.8 -> 422.6 mm
- net Net-(LD0,4-Pad4): track 411.5 -> 419.1 mm
- net Net-(LD0,2-Pad4): track 435.5 -> 438.7 mm
- net Net-(LD0,5-Pad5): track 462.1 -> 464.5 mm
- net Net-(LD0,1-Pad4): track 437.3 -> 439.4 mm
- net Net-(LD0,1-Pad5): track 444.9 -> 447.0 mm
- net Net-(LD0,5-Pad4): track 460.8 -> 462.5 mm
- net KEY_ROW3: track 476.7 -> 475.9 mm, vias 1 -> 2
- net Net-(LD0,2-Pad5): track 437.5 -> 438.2 mm
- net Net-(J1-Pad34): vias 0 -> 1
- net Net-(J1-Pad33): vias 0 -> 1
- net Net-(J1-Pad32): vias 0 -> 1
- net Net-(J1-Pad31): vias 0 -> 1
- net LED_SDA_STATUS0: vias 0 -> 1
- net LED_SDA_ROW0: vias 0 -> 1
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