File: KiCAD/Mainboard/RedPyKeeb_mainboard.kicad_pcb (KiCad board)
At the start: 4 copper layers, 440.7 x 154.9 mm, 333 parts, among them J1 Conn_02x20_Top_Bottom

Commit message: Fix issues found with MCU and mainboard PCBs. Adding whatever fiddling I had with firmware.
Parts:
- removed the C6 at (430.3, 25.4) (x2)
- added C6: EEE-FN1C102UV, Capacitor_SMD:CP_Elec_10x10, F.Cu at (430.3, 25.4)
- added C6: EEE-FN1C102UV, Capacitor_SMD:CP_Elec_10x10, B.Cu at (430.3, 25.4)
- moved K8,0 5.52 mm to (206.4, 55.6)
- moved LD8,0 5.52 mm to (206.6, 48.6)
- moved D8,0 5.52 mm to (198.6, 56.8)
- moved K7,0 5.27 mm to (187.3, 55.6)
- moved D7,0 5.27 mm to (179.5, 56.8)
- moved LD7,0 5.27 mm to (187.5, 48.6)
- moved D6,0 5.01 mm to (160.5, 56.8)
- moved K6,0 5.01 mm to (168.3, 55.6)
- moved LD6,0 5.01 mm to (168.5, 48.6)
- moved D12,0 4.92 mm to (283.5, 56.8)
- moved K12,0 4.92 mm to (291.3, 55.6)
- moved LD12,0 4.92 mm to (291.5, 48.6)
- moved D11,5 4.80 mm to (281.9, 157.6)
- moved K11,5 4.80 mm to (289.7, 156.4)
- moved LD11,5 4.80 mm to (289.7, 149.5)
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Routing:
- net KEY_ROW0: track 554.9 -> 491.1 mm, vias 3 -> 2
- net KEY_ROW1: track 565.7 -> 524.5 mm
- net KEY_ROW5: track 580.5 -> 554.1 mm, vias 4 -> 2
- net Net-(LD0,5-Pad5): track 464.5 -> 439.8 mm
- net Net-(LD0,5-Pad4): track 462.5 -> 438.8 mm
- net KEY_ROW4: track 535.7 -> 513.3 mm
- net Net-(LD0,4-Pad5): track 422.6 -> 406.5 mm
- net KEY_ROW6: track 317.4 -> 302.0 mm, vias 4 -> 2
- net Net-(LD0,2-Pad4): track 438.7 -> 424.8 mm
- net Net-(LD0,4-Pad4): track 419.1 -> 406.1 mm
- net KEY_COL11: track 294.2 -> 281.7 mm
- net Net-(LD0,2-Pad5): track 438.2 -> 425.7 mm
- net LED_SDA_STATUS0: track 156.0 -> 143.7 mm, vias 1 -> 3
- net KEY_COL5: track 350.6 -> 340.6 mm
- net Net-(LD0,1-Pad5): track 447.0 -> 437.1 mm
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Other:
- board size 440.7 x 154.9 mm -> 432 x 151 mm
